Commit message: messing with urdf

File: legged_perceptive_description/urdf/gazebo_d400.xacro (robot description, xacro)
@@ -19,4 +19,5 @@
             <!--<max_vel>0.01</max_vel>
             <min_depth>0</min_depth>-->
+            <!-- Color Camera Sensor -->
             <sensor name="${camera_name}color" type="camera">
                 <camera name="${camera_name}">
@@ -41,4 +42,5 @@
                 <visualize>1</visualize>
             </sensor>
+            <!-- Infrared Cameras -->
             <sensor name="${camera_name}ired1" type="camera">
                 <camera name="${camera_name}">
@@ -85,10 +87,12 @@
                 <visualize>0</visualize>
             </sensor>
+            <!-- Depth Sensor with Reduced Resolution -->
             <sensor name="${camera_name}depth" type="depth">
                 <camera name="${camera_name}">
                     <horizontal_fov>${85.2*deg_to_rad}</horizontal_fov>
                     <image>
-                        <width>1280</width>
-                        <height>720</height>
+                        <!-- Reduced resolution from 1280x720 to 640x360 -->
+                        <width>320</width>
+                        <height>180</height>
                     </image>
                     <clip>
@@ -103,4 +107,5 @@
                 </camera>
                 <always_on>1</always_on>
+                <!-- Optionally reduce update rate if needed -->
                 <update_rate>10</update_rate>
                 <visualize>0</visualize>

File: legged_perceptive_description/urdf/livox_mid360.xacro (robot description, xacro)
@@ -16,17 +16,20 @@
     </inertial>
   </xacro:macro>
-  <!-- Updated Livox Mid360 sensor macro with matching naming -->
+  <!-- Livox Mid360 sensor macro with unique naming -->
   <xacro:macro name="Livox_Mid360" params="name parent *origin ros_topic:=livox visualize:=True update_rate:=10 resolution:=0.002 noise_mean:=0.0 noise_stddev:=0.01">
-    <!-- Sensor link with physical and visual details -->
-    <link name="${name}">
+    <!-- Sensor Link with Unique Name -->
+    <link name="${name}_link">
       <inertial>
         <origin rpy="0 0 0" xyz="0 0 -0.0076"/>
         <mass value="0.270"/>
         <inertia
-          ixx="${(2*0.270)/5.0*(0.022*0.022)}" ixy="0.0" ixz="0.0"
-          iyy="${(2*0.270)/5.0*(0.022*0.022)}" iyz="0.0"
-          izz="${(2*0.270)/5.0*(0.022*0.022)}"/>
+          ixx="${(2 * 0.270) / 5.0 * (0.022 * 0.022)}"
+          ixy="0.0"
+          ixz="0.0"
+          iyy="${(2 * 0.270) / 5.0 * (0.022 * 0.022)}"
+          iyz="0.0"
+          izz="${(2 * 0.270) / 5.0 * (0.022 * 0.022)}"/>
       </inertial>
-      <!-- Visual using sphere -->
+      <!-- Visual using Sphere -->
       <visual>
         <origin rpy="0 0 0" xyz="0 0 -0.0076"/>
@@ -34,7 +37,10 @@
           <sphere radius="0.022"/>
         </geometry>
-        <color rgba="0.0 0.0 0.5 0.5"/>
+        <material>
+          <color rgba="0.0 0.0 0.5 0.5"/>
+        </material>
       </visual>
-      <!-- Collision elements from the old macro -->
+      <!-- Optional: Add Collision Elements Here If Needed -->
+      <!--
       <collision>
         <origin xyz="0 0 0.027" rpy="0 0 0"/>
@@ -43,50 +49,21 @@
         </geometry>
       </collision>
-      <collision>
-        <origin xyz="0 0.041 0.007" rpy="-1.04 0 0"/>
-        <geometry>
-          <box size="0.003 0.055 0.024"/>
-        </geometry>
-      </collision>
-      <collision>
-        <origin xyz="0 -0.041 0.007" rpy="1.04 0 0"/>
-        <geometry>
-          <box size="0.003 0.055 0.024"/>
-        </geometry>
-      </collision>
-      <collision>
-        <origin xyz="0 0 0.027" rpy="0 0 0"/>
-        <geometry>
-          <box size="0.067 0.003 0.0165"/>
-        </geometry>
-      </collision>
-      <collision>
-        <origin xyz="0.041 0 0.007" rpy="0 1.04 0"/>
-        <geometry>
-          <box size="0.055 0.003 0.024"/>
-        </geometry>
-      </collision>
-      <collision>
-        <origin xyz="-0.041 0 0.007" rpy="0 -1.04 0"/>
-        <geometry>
-          <box size="0.055 0.003 0.024"/>
-        </geometry>
-      </collision>
+      -->
     </link>
-    <!-- Joint to attach sensor to parent link -->
-    <joint name="${name}_fixed" type="fixed">
-      <xacro:insert_block name="origin"/>
+    <!-- Fixed Joint to Attach Sensor to Parent Link -->
+    <joint name="${name}_fixed_joint" type="fixed">
+      <origin xyz="0 0 0" rpy="0 0 0"/> <!-- Replace with actual origin if different -->
       <parent link="${parent}"/>
-      <child link="${name}"/>
+      <child link="${name}_link"/>
     </joint>
-    <!-- Gazebo sensor plugin for visualization and sensor properties -->
-    <gazebo reference="${name}">
+    <!-- Gazebo Sensor Plugin for Visualization and Sensor Properties -->
+    <gazebo reference="${name}_link">
       <self_collide>1</self_collide>
       <material>Gazebo/Blue</material>
-      <sensor type="ray" name="${name}">
+      <sensor type="ray" name="${name}_sensor">
         <pose>0 0 0 0 0 0</pose>
         <visualize>${visualize}</visualize>
         <update_rate>${update_rate}</update_rate>
-        <plugin name="gazebo_ros_laser_controller" filename="liblivox_laser_simulation.so">
+        <plugin name="${name}_gazebo_plugin" filename="liblivox_laser_simulation.so">
           <ray>
             <scan>
@@ -95,11 +72,11 @@
                 <resolution>1</resolution>
                 <min_angle>0</min_angle>
-                <max_angle>${2*M_PI}</max_angle>
+                <max_angle>${2 * M_PI}</max_angle>
               </horizontal>
               <vertical>
                 <samples>360</samples>
                 <resolution>1</resolution>
-                <min_angle>${-7.22/180*M_PI}</min_angle>
-                <max_angle>${55.22/180*M_PI}</max_angle>
+                <min_angle>${-7.22 / 180 * M_PI}</min_angle>
+                <max_angle>${55.22 / 180 * M_PI}</max_angle>
               </vertical>
             </scan>

File: legged_perceptive_description/urdf/robot.xacro (robot description, xacro)
@@ -6,5 +6,6 @@
     <!-- <xacro:include filename="$(find legged_perceptive_description)/urdf/sensor_t265.xacro"/> -->
     <!-- <xacro:include filename="$(find legged_perceptive_description)/urdf/mid360.xacro"/> -->
-    <xacro:include filename="$(find legged_perceptive_description)/urdf/livox_mid360.xacro"/>
+    <!-- <xacro:include filename="$(find legged_perceptive_description)/urdf/livox_mid360.xacro"/> -->
+    <xacro:include filename="$(find legged_perceptive_description)/urdf/livox_mid360_2.xacro"/>
     <xacro:sensor_d435 name="front_camera" topics_ns="front_camera" parent="base">
         <origin xyz="0.31 -0.0 0.11" rpy="3.141 0.38 0"/>
@@ -13,9 +14,10 @@
         <origin xyz="0.16 0 0.085" rpy="0 -1.04 0"/>
     </xacro:sensor_t265> -->
-    <xacro:Livox_Mid360 name="livox_right" parent="base" ros_topic="/livox/lidar_192_168_8_101">
+    <!-- <xacro:Livox_Mid360 name="livox_right" parent="base" ros_topic="/livox/lidar_192_168_8_101">
         <origin xyz="0.365 -0.068 -0.030" rpy="-2.59 1.03 3.09"/>
-    </xacro:Livox_Mid360>
-    <xacro:Livox_Mid360 name="livox_left" parent="base" ros_topic="/livox/lidar_192_168_8_102">
+    </xacro:Livox_Mid360> -->
+    <!-- <xacro:Livox_Mid360 name="livox_left" parent="base" ros_topic="/livox/lidar_192_168_8_102">
         <origin xyz="0.365 0.068 -0.030" rpy="2.59 1.03 -3.09"/>
-    </xacro:Livox_Mid360>
+    </xacro:Livox_Mid360> -->
+    <xacro:Livox_Mid_gazebo_sensor/>
 </robot>

File: legged_perceptive_description/urdf/sensor_d435.xacro (robot description, xacro)
@@ -40,6 +40,6 @@
                 <origin xyz="${d435_cam_mount_from_center_offset} ${-d435_cam_depth_py} 0" rpy="${M_PI/2} 0 ${M_PI/2}"/>
                 <geometry>
-                    <!-- <box size="${d435_cam_width} ${d435_cam_height} ${d435_cam_depth}"/> -->
-                    <mesh filename="package://realsense2_description/meshes/d435.dae"/>
+                    <box size="${d435_cam_width} ${d435_cam_height} ${d435_cam_depth}"/>
+                    <!-- <mesh filename="package://realsense2_description/meshes/d435.dae"/> -->
                     <!--<mesh filename="package://realsense2_description/meshes/d435/d435.dae" />-->
                 </geometry>
