Commit message: insert_block

File: legged_perceptive_description/urdf/livox_mid360.xacro (robot description, xacro)
@@ -44,48 +44,11 @@
             </geometry>
             <color rgba="0.0 0.0 0.5 0.5"/>
-    </visual>
-      <!-- Collisions for more accurate simulation -->
-      <collision>
-        <origin xyz="0 0 0.027" rpy="0 0 0"/>
-        <geometry>
-          <box size="0.003 0.067 0.0165"/>
-        </geometry>
-      </collision>
-      <collision>
-        <origin xyz="0 0.041 0.007" rpy="-1.04 0 0"/>
-        <geometry>
-          <box size="0.003 0.055 0.024"/>
-        </geometry>
-      </collision>
-      <collision>
-        <origin xyz="0 -0.041 0.007" rpy="1.04 0 0"/>
-        <geometry>
-          <box size="0.003 0.055 0.024"/>
-        </geometry>
-      </collision>
-      <collision>
-        <origin xyz="0 0 0.027" rpy="0 0 0"/>
-        <geometry>
-          <box size="0.067 0.003 0.0165"/>
-        </geometry>
-      </collision>
-      <collision>
-        <origin xyz="0.041 0 0.007" rpy="0 1.04 0"/>
-        <geometry>
-          <box size="0.055 0.003 0.024"/>
-        </geometry>
-      </collision>
-      <collision>
-        <origin xyz="-0.041 0 0.007" rpy="0 -1.04 0"/>
-        <geometry>
-          <box size="0.055 0.003 0.024"/>
-        </geometry>
-      </collision>
+      </visual>
     </link>
     <!-- Joint to attach sensor to parent link -->
     <joint name="${name}_to_${name}_base_joint" type="fixed">
-      <parent link="${parent}"/>
-      <child link="${name}_base"/>
-      <origin rpy="0 0 0" xyz="0.0 1.0 0.2"/>
+        <parent link="${parent}"/>
+        <child link="${name}_base"/>
+        <xacro:insert_block name="origin"/>
     </joint>
     <!-- Gazebo sensor plugin for visualization and sensor properties -->

Commit message: origin name origin

File: legged_perceptive_description/urdf/livox_mid360.xacro (robot description, xacro)
@@ -48,7 +48,7 @@
     <!-- Joint to attach sensor to parent link -->
     <joint name="${name}_to_${name}_base_joint" type="fixed">
+        <xacro:insert_block name="origin"/>
         <parent link="${parent}"/>
         <child link="${name}_base"/>
-        <xacro:insert_block name="origin"/>
     </joint>
     <!-- Gazebo sensor plugin for visualization and sensor properties -->

File: legged_perceptive_description/urdf/robot.xacro (robot description, xacro)
@@ -14,8 +14,8 @@
     </xacro:sensor_t265> -->
     <xacro:Livox_Mid360 name="livox_right" parent="base">
-        <origin xyz="0.365 -0.068 -0.030" rpy="-2.59 1.03 3.09"/>
+        <origin xacro:name="origin" xyz="0.365 -0.068 -0.030" rpy="-2.59 1.03 3.09"/>
     </xacro:Livox_Mid360>
     <xacro:Livox_Mid360 name="livox_left" parent="base">
-        <origin xyz="0.365 0.068 -0.030" rpy="2.59 1.03 -3.09"/>
+        <origin xacro:name="origin" xyz="0.365 0.068 -0.030" rpy="2.59 1.03 -3.09"/>
     </xacro:Livox_Mid360>
 </robot>

Commit message: test

File: legged_perceptive_description/urdf/livox_mid360.xacro (robot description, xacro)
@@ -18,5 +18,5 @@
   </xacro:macro>
   <!-- Define the main Livox Mid360 sensor macro -->
-  <xacro:macro name="Livox_Mid360" params="name parent visualize:=True update_rate:=10 resolution:=0.002 noise_mean:=0.0 noise_stddev:=0.01">
+  <xacro:macro name="Livox_Mid360" params="name parent visualize:=True update_rate:=10 resolution:=0.002 noise_mean:=0.0 noise_stddev:=0.01 *origin">
     <!-- Sensor base link with physical and visual details -->
     <link name="${name}_base">
@@ -29,26 +29,20 @@
           izz="${(2*0.270)/5.0*(0.022*0.022)}"/>
       </inertial>
-      <!-- Visual using mesh -->
-      <!-- <visual>
-        <origin xyz="0.00 0 0.0" rpy="0 0 0"/>
+      <!-- Visual using sphere -->
+      <visual>
+        <origin rpy="0 0 0" xyz="0 0 -0.0076"/>
         <geometry>
-          <mesh filename="package://livox_laser_simulation/meshes/livox_mid40.dae"/>
+          <sphere radius="0.022"/>
         </geometry>
         <color rgba="0.0 0.0 0.5 0.5"/>
-      </visual> -->
-      <!-- Visual using sphere -->
-      <visual>
-            <origin rpy="0 0 0" xyz="0 0 -0.0076"/>
-            <geometry>
-                <sphere radius="0.022"/>
-            </geometry>
-            <color rgba="0.0 0.0 0.5 0.5"/>
       </visual>
     </link>
     <!-- Joint to attach sensor to parent link -->
     <joint name="${name}_to_${name}_base_joint" type="fixed">
+      <parent link="${parent}"/>
+      <child link="${name}_base"/>
+      <xacro:if value="$(has_block origin)">
         <xacro:insert_block name="origin"/>
-        <parent link="${parent}"/>
-        <child link="${name}_base"/>
+      </xacro:if>
     </joint>
     <!-- Gazebo sensor plugin for visualization and sensor properties -->
@@ -94,3 +88,12 @@
     </gazebo>
   </xacro:macro>
+  <!-- Instantiate the macro with origin blocks -->
+  <!-- <xacro:Livox_Mid360 name="livox_right" parent="base">
+    <origin xyz="0.365 -0.068 -0.030" rpy="-2.59 1.03 3.09"/>
+  </xacro:Livox_Mid360>
+  <xacro:Livox_Mid360 name="livox_left" parent="base">
+    <origin xyz="0.365 0.068 -0.030" rpy="2.59 1.03 -3.09"/>
+  </xacro:Livox_Mid360>
+  <!-- If you want to instantiate without an origin, ensure the macro handles it -->
+  <xacro:Livox_Mid360 name="livox_center" parent="base_link"/> -->
 </robot>

Commit message: back

File: legged_perceptive_description/urdf/livox_mid360.xacro (robot description, xacro)
@@ -18,5 +18,5 @@
   </xacro:macro>
   <!-- Define the main Livox Mid360 sensor macro -->
-  <xacro:macro name="Livox_Mid360" params="name parent visualize:=True update_rate:=10 resolution:=0.002 noise_mean:=0.0 noise_stddev:=0.01 *origin">
+  <xacro:macro name="Livox_Mid360" params="name parent visualize:=True update_rate:=10 resolution:=0.002 noise_mean:=0.0 noise_stddev:=0.01">
     <!-- Sensor base link with physical and visual details -->
     <link name="${name}_base">
@@ -29,20 +29,26 @@
           izz="${(2*0.270)/5.0*(0.022*0.022)}"/>
       </inertial>
+      <!-- Visual using mesh -->
+      <!-- <visual>
+        <origin xyz="0.00 0 0.0" rpy="0 0 0"/>
+        <geometry>
+          <mesh filename="package://livox_laser_simulation/meshes/livox_mid40.dae"/>
+        </geometry>
+        <color rgba="0.0 0.0 0.5 0.5"/>
+      </visual> -->
       <!-- Visual using sphere -->
       <visual>
-        <origin rpy="0 0 0" xyz="0 0 -0.0076"/>
-        <geometry>
-          <sphere radius="0.022"/>
-        </geometry>
-        <color rgba="0.0 0.0 0.5 0.5"/>
+            <origin rpy="0 0 0" xyz="0 0 -0.0076"/>
+            <geometry>
+                <sphere radius="0.022"/>
+            </geometry>
+            <color rgba="0.0 0.0 0.5 0.5"/>
       </visual>
     </link>
     <!-- Joint to attach sensor to parent link -->
     <joint name="${name}_to_${name}_base_joint" type="fixed">
-      <parent link="${parent}"/>
-      <child link="${name}_base"/>
-      <xacro:if value="$(has_block origin)">
         <xacro:insert_block name="origin"/>
-      </xacro:if>
+        <parent link="${parent}"/>
+        <child link="${name}_base"/>
     </joint>
     <!-- Gazebo sensor plugin for visualization and sensor properties -->
@@ -88,12 +94,3 @@
     </gazebo>
   </xacro:macro>
-  <!-- Instantiate the macro with origin blocks -->
-  <!-- <xacro:Livox_Mid360 name="livox_right" parent="base">
-    <origin xyz="0.365 -0.068 -0.030" rpy="-2.59 1.03 3.09"/>
-  </xacro:Livox_Mid360>
-  <xacro:Livox_Mid360 name="livox_left" parent="base">
-    <origin xyz="0.365 0.068 -0.030" rpy="2.59 1.03 -3.09"/>
-  </xacro:Livox_Mid360>
-  <!-- If you want to instantiate without an origin, ensure the macro handles it -->
-  <xacro:Livox_Mid360 name="livox_center" parent="base_link"/> -->
 </robot>

Commit message: testin

File: legged_perceptive_description/urdf/livox_mid360.xacro (robot description, xacro)
@@ -29,14 +29,6 @@
           izz="${(2*0.270)/5.0*(0.022*0.022)}"/>
       </inertial>
-      <!-- Visual using mesh -->
+      <!-- Visual using sphere -->
       <!-- <visual>
-        <origin xyz="0.00 0 0.0" rpy="0 0 0"/>
-        <geometry>
-          <mesh filename="package://livox_laser_simulation/meshes/livox_mid40.dae"/>
-        </geometry>
-        <color rgba="0.0 0.0 0.5 0.5"/>
-      </visual> -->
-      <!-- Visual using sphere -->
-      <visual>
             <origin rpy="0 0 0" xyz="0 0 -0.0076"/>
             <geometry>
@@ -44,5 +36,5 @@
             </geometry>
             <color rgba="0.0 0.0 0.5 0.5"/>
-      </visual>
+      </visual> -->
     </link>
     <!-- Joint to attach sensor to parent link -->

File: legged_perceptive_description/urdf/robot.xacro (robot description, xacro)
@@ -14,8 +14,8 @@
     </xacro:sensor_t265> -->
     <xacro:Livox_Mid360 name="livox_right" parent="base">
-        <origin xacro:name="origin" xyz="0.365 -0.068 -0.030" rpy="-2.59 1.03 3.09"/>
+        <origin xyz="0.365 -0.068 -0.030" rpy="-2.59 1.03 3.09"/>
     </xacro:Livox_Mid360>
     <xacro:Livox_Mid360 name="livox_left" parent="base">
-        <origin xacro:name="origin" xyz="0.365 0.068 -0.030" rpy="2.59 1.03 -3.09"/>
+        <origin xyz="0.365 0.068 -0.030" rpy="2.59 1.03 -3.09"/>
     </xacro:Livox_Mid360>
 </robot>

Commit message: include in params list!

File: legged_perceptive_description/urdf/livox_mid360.xacro (robot description, xacro)
@@ -18,5 +18,5 @@
   </xacro:macro>
   <!-- Define the main Livox Mid360 sensor macro -->
-  <xacro:macro name="Livox_Mid360" params="name parent visualize:=True update_rate:=10 resolution:=0.002 noise_mean:=0.0 noise_stddev:=0.01">
+  <xacro:macro name="Livox_Mid360" params="name parent *origin visualize:=True update_rate:=10 resolution:=0.002 noise_mean:=0.0 noise_stddev:=0.01">
     <!-- Sensor base link with physical and visual details -->
     <link name="${name}_base">

Commit message: re-enable visual

File: legged_perceptive_description/urdf/livox_mid360.xacro (robot description, xacro)
@@ -30,5 +30,5 @@
       </inertial>
       <!-- Visual using sphere -->
-      <!-- <visual>
+      <visual>
             <origin rpy="0 0 0" xyz="0 0 -0.0076"/>
             <geometry>
@@ -36,5 +36,5 @@
             </geometry>
             <color rgba="0.0 0.0 0.5 0.5"/>
-      </visual> -->
+      </visual>
     </link>
     <!-- Joint to attach sensor to parent link -->

Commit message: topics

File: legged_perceptive_description/urdf/livox_mid360.xacro (robot description, xacro)
@@ -5,5 +5,4 @@
   <xacro:property name="laser_min_range" value="0.1"/>
   <xacro:property name="laser_max_range" value="200.0"/>
-  <xacro:property name="ros_topic" value="scan"/>
   <xacro:property name="samples" value="24000"/>
   <xacro:property name="downsample" value="1"/>
@@ -18,5 +17,5 @@
   </xacro:macro>
   <!-- Define the main Livox Mid360 sensor macro -->
-  <xacro:macro name="Livox_Mid360" params="name parent *origin visualize:=True update_rate:=10 resolution:=0.002 noise_mean:=0.0 noise_stddev:=0.01">
+  <xacro:macro name="Livox_Mid360" params="name parent *origin ros_topic:=livox visualize:=True update_rate:=10 resolution:=0.002 noise_mean:=0.0 noise_stddev:=0.01">
     <!-- Sensor base link with physical and visual details -->
     <link name="${name}_base">

File: legged_perceptive_description/urdf/robot.xacro (robot description, xacro)
@@ -13,8 +13,8 @@
         <origin xyz="0.16 0 0.085" rpy="0 -1.04 0"/>
     </xacro:sensor_t265> -->
-    <xacro:Livox_Mid360 name="livox_right" parent="base">
+    <xacro:Livox_Mid360 name="livox_right" parent="base" ros_topic="/livox/lidar_192_168_8_101">
         <origin xyz="0.365 -0.068 -0.030" rpy="-2.59 1.03 3.09"/>
     </xacro:Livox_Mid360>
-    <xacro:Livox_Mid360 name="livox_left" parent="base">
+    <xacro:Livox_Mid360 name="livox_left" parent="base" ros_topic="/livox/lidar_192_168_8_102">
         <origin xyz="0.365 0.068 -0.030" rpy="2.59 1.03 -3.09"/>
     </xacro:Livox_Mid360>

Commit message: naming

File: legged_perceptive_description/urdf/livox_mid360.xacro (robot description, xacro)
@@ -41,8 +41,8 @@
         <xacro:insert_block name="origin"/>
         <parent link="${parent}"/>
-        <child link="${name}_base"/>
+        <child link="${name}"/>
     </joint>
     <!-- Gazebo sensor plugin for visualization and sensor properties -->
-    <gazebo reference="${name}_base">
+    <gazebo reference="${name}">
       <sensor type="ray" name="${name}">
         <pose>0 0 0 0 0 0</pose>

Commit message: naming etc

File: legged_perceptive_description/urdf/livox_mid360.xacro (robot description, xacro)
@@ -16,8 +16,8 @@
     </inertial>
   </xacro:macro>
-  <!-- Define the main Livox Mid360 sensor macro -->
+  <!-- Updated Livox Mid360 sensor macro with matching naming -->
   <xacro:macro name="Livox_Mid360" params="name parent *origin ros_topic:=livox visualize:=True update_rate:=10 resolution:=0.002 noise_mean:=0.0 noise_stddev:=0.01">
-    <!-- Sensor base link with physical and visual details -->
-    <link name="${name}_base">
+    <!-- Sensor link with physical and visual details -->
+    <link name="${name}">
       <inertial>
         <origin rpy="0 0 0" xyz="0 0 -0.0076"/>
@@ -30,19 +30,58 @@
       <!-- Visual using sphere -->
       <visual>
-            <origin rpy="0 0 0" xyz="0 0 -0.0076"/>
-            <geometry>
-                <sphere radius="0.022"/>
-            </geometry>
-            <color rgba="0.0 0.0 0.5 0.5"/>
+        <origin rpy="0 0 0" xyz="0 0 -0.0076"/>
+        <geometry>
+          <sphere radius="0.022"/>
+        </geometry>
+        <color rgba="0.0 0.0 0.5 0.5"/>
       </visual>
+      <!-- Collision elements from the old macro -->
+      <collision>
+        <origin xyz="0 0 0.027" rpy="0 0 0"/>
+        <geometry>
+          <box size="0.003 0.067 0.0165"/>
+        </geometry>
+      </collision>
+      <collision>
+        <origin xyz="0 0.041 0.007" rpy="-1.04 0 0"/>
+        <geometry>
+          <box size="0.003 0.055 0.024"/>
+        </geometry>
+      </collision>
+      <collision>
+        <origin xyz="0 -0.041 0.007" rpy="1.04 0 0"/>
+        <geometry>
+          <box size="0.003 0.055 0.024"/>
+        </geometry>
+      </collision>
+      <collision>
+        <origin xyz="0 0 0.027" rpy="0 0 0"/>
+        <geometry>
+          <box size="0.067 0.003 0.0165"/>
+        </geometry>
+      </collision>
+      <collision>
+        <origin xyz="0.041 0 0.007" rpy="0 1.04 0"/>
+        <geometry>
+          <box size="0.055 0.003 0.024"/>
+        </geometry>
+      </collision>
+      <collision>
+        <origin xyz="-0.041 0 0.007" rpy="0 -1.04 0"/>
+        <geometry>
+          <box size="0.055 0.003 0.024"/>
+        </geometry>
+      </collision>
     </link>
     <!-- Joint to attach sensor to parent link -->
-    <joint name="${name}_to_${name}_base_joint" type="fixed">
-        <xacro:insert_block name="origin"/>
-        <parent link="${parent}"/>
-        <child link="${name}"/>
+    <joint name="${name}_fixed" type="fixed">
+      <xacro:insert_block name="origin"/>
+      <parent link="${parent}"/>
+      <child link="${name}"/>
     </joint>
     <!-- Gazebo sensor plugin for visualization and sensor properties -->
     <gazebo reference="${name}">
+      <self_collide>1</self_collide>
+      <material>Gazebo/Blue</material>
       <sensor type="ray" name="${name}">
         <pose>0 0 0 0 0 0</pose>

Commit message: sim lidar

File: legged_perceptive_description/urdf/livox_mid360.xacro (robot description, xacro)
@@ -17,5 +17,5 @@
   </xacro:macro>
   <!-- Livox Mid360 sensor macro with unique naming -->
-  <xacro:macro name="Livox_Mid360" params="name parent *origin ros_topic:=livox visualize:=True update_rate:=10 resolution:=0.002 noise_mean:=0.0 noise_stddev:=0.01">
+  <xacro:macro name="Livox_Mid360" params="name parent *origin ros_topic:=livox visualize:=False update_rate:=10 resolution:=0.002 noise_mean:=0.0 noise_stddev:=0.01">
     <!-- Sensor Link with Unique Name -->
     <link name="${name}_link">
@@ -65,5 +65,5 @@
         <visualize>${visualize}</visualize>
         <update_rate>${update_rate}</update_rate>
-        <plugin name="${name}_gazebo_plugin" filename="liblivox_laser_simulation.so">
+        <plugin name="gazebo_ros_laser_controller" filename="liblivox_laser_simulation.so">
           <ray>
             <scan>
@@ -75,5 +75,5 @@
               </horizontal>
               <vertical>
-                <samples>360</samples>
+                <samples>50</samples>
                 <resolution>1</resolution>
                 <min_angle>${-7.22 / 180 * M_PI}</min_angle>
@@ -95,5 +95,7 @@
           <samples>${samples}</samples>
           <downsample>${downsample}</downsample>
-          <csv_file_name>package://livox_laser_simulation/scan_mode/mid360.csv</csv_file_name>
+          <publish_pointcloud_type>2</publish_pointcloud_type>
+          <frameName>${name}_link</frameName>
+          <csv_file_name>mid360-real-centr.csv</csv_file_name>
           <ros_topic>${ros_topic}</ros_topic>
         </plugin>

File: legged_perceptive_description/urdf/robot.xacro (robot description, xacro)
@@ -6,16 +6,14 @@
     <!-- <xacro:include filename="$(find legged_perceptive_description)/urdf/sensor_t265.xacro"/> -->
     <xacro:include filename="$(find legged_perceptive_description)/urdf/sensor_mid360.xacro"/>
+    <!-- <xacro:include filename="$(find legged_perceptive_description)/urdf/livox_mid360.xacro"/> -->
     <!-- <xacro:sensor_d435 name="front_camera" topics_ns="front_camera" parent="base">
            <origin xyz="0.31 -0.0 0.11" rpy="3.141 0.38 0"/>
-      </xacro:sensor_d435> -->
+    </xacro:sensor_d435> -->
     <!-- <xacro:sensor_t265 name="tracking_camera" topics_ns="tracking_camera" parent="base">
         <origin xyz="0.16 0 0.085" rpy="0 -1.04 0"/>
     </xacro:sensor_t265> -->
-    <!-- <xacro:Livox_Mid360 name="livox_right" parent="base" ros_topic="/livox/lidar_192_168_8_101">
-        <origin xyz="0.365 -0.068 -0.030" rpy="-2.59 1.03 3.09"/>
-    </xacro:mid360> -->
-    <xacro:sensor_mid360 name="livox_front" topics_ns="lidar_192_168_8_101" parent="base" xyz="0.25 0 0.150" rpy="0 0.5 0" sim="true"/>
-    <!-- <xacro:Livox_Mid360 name="livox_left" parent="base" ros_topic="/livox/lidar_192_168_8_102">
-        <origin xyz="0.365 0.068 -0.030" rpy="2.59 1.03 -3.09"/>
-    </xacro:Livox_Mid360> -->
+    <xacro:sensor_mid360 name="livox_front" topics_ns="lidar_192_168_1_105" parent="base" xyz="0.25 0 0.350" rpy="0 0.5 0" sim="true"/>
+    <!-- <xacro:Livox_Mid_gazebo_sensor name="livox_front" parent="base" ros_topic="/livox/lidar_192_168_1_105">
+        <origin xyz="0.25 0 0.150" rpy="0 0.5 0"/>
+    </xacro:Livox_Mid_gazebo_sensor> -->
 </robot>

File: legged_perceptive_description/urdf/sensor_mid360.xacro (robot description, xacro)
@@ -18,7 +18,7 @@
             <visual>
                 <origin xyz="0 0 0" rpy="0 0 0"/>
-                <geometry>
+                <!-- <geometry>
                     <mesh filename="file://$(find livox_laser_simulation)/meshes/livox_mid-360-90x.dae" scale="1 1 1"/>
-                </geometry>
+                </geometry> -->
                 <material name="${name}_material"/>
             </visual>
@@ -47,5 +47,4 @@
             <gazebo reference="${name}_sensor_frame">
                 <sensor type="ray" name="${name}_laser_livox">
-                    <pose>${xyz} ${rpy}</pose>
                     <visualize>true</visualize>
                     <always_on>true</always_on>
