Commit message: working lidar in elevation mapping

File: legged_perceptive_description/urdf/robot.xacro (robot description, xacro)
@@ -5,10 +5,8 @@
     <xacro:include filename="$(find legged_perceptive_description)/urdf/sensor_d435.xacro"/>
     <!-- <xacro:include filename="$(find legged_perceptive_description)/urdf/sensor_t265.xacro"/> -->
-    <!-- <xacro:include filename="$(find legged_perceptive_description)/urdf/mid360.xacro"/> -->
-    <!-- <xacro:include filename="$(find legged_perceptive_description)/urdf/livox_mid360.xacro"/> -->
-    <xacro:include filename="$(find legged_perceptive_description)/urdf/livox_mid360_2.xacro"/>
-    <xacro:sensor_d435 name="front_camera" topics_ns="front_camera" parent="base">
-        <origin xyz="0.31 -0.0 0.11" rpy="3.141 0.38 0"/>
-    </xacro:sensor_d435>
+    <xacro:include filename="$(find legged_perceptive_description)/urdf/sensor_mid360.xacro"/>
+    <!-- <xacro:sensor_d435 name="front_camera" topics_ns="front_camera" parent="base">
+           <origin xyz="0.31 -0.0 0.11" rpy="3.141 0.38 0"/>
+      </xacro:sensor_d435> -->
     <!-- <xacro:sensor_t265 name="tracking_camera" topics_ns="tracking_camera" parent="base">
         <origin xyz="0.16 0 0.085" rpy="0 -1.04 0"/>
@@ -16,5 +14,6 @@
     <!-- <xacro:Livox_Mid360 name="livox_right" parent="base" ros_topic="/livox/lidar_192_168_8_101">
         <origin xyz="0.365 -0.068 -0.030" rpy="-2.59 1.03 3.09"/>
-    </xacro:Livox_Mid360> -->
+    </xacro:mid360> -->
+    <xacro:sensor_mid360 name="livox_front" topics_ns="lidar_192_168_8_101" parent="base" xyz="0.25 0 0.150" rpy="0 0.5 0" sim="true"/>
     <!-- <xacro:Livox_Mid360 name="livox_left" parent="base" ros_topic="/livox/lidar_192_168_8_102">
         <origin xyz="0.365 0.068 -0.030" rpy="2.59 1.03 -3.09"/>

Commit message: adding back camera

File: legged_perceptive_description/urdf/robot.xacro (robot description, xacro)
@@ -7,7 +7,7 @@
     <xacro:include filename="$(find legged_perceptive_description)/urdf/sensor_mid360.xacro"/>
     <xacro:include filename="$(find legged_perceptive_description)/urdf/nuc_and_lidar/nuc_and_lidar.xacro"/>
-    <!-- <xacro:sensor_d435 name="front_camera" topics_ns="front_camera" parent="base">
-           <origin xyz="0.31 -0.0 0.11" rpy="3.141 0.38 0"/>
-      </xacro:sensor_d435> -->
+    <xacro:sensor_d435 name="front_camera" topics_ns="front_camera" parent="base" sim="true">
+           <origin xyz="0.33 -0.0 0.09" rpy="0 0.83 0"/>
+      </xacro:sensor_d435>
     <!-- <xacro:sensor_t265 name="tracking_camera" topics_ns="tracking_camera" parent="base">
         <origin xyz="0.16 0 0.085" rpy="0 -1.04 0"/>

File: legged_perceptive_description/urdf/sensor_d435.xacro (robot description, xacro)
@@ -112,6 +112,5 @@
             </joint>
             <link name="${name}_color_optical_frame"/>
-            <xacro:include filename="$(find legged_perceptive_description)/urdf/gazebo_d400.xacro"/>
-            <!-- Realsense Gazebo Plugin -->
+            <!-- <xacro:include filename="$(find legged_perceptive_description)/urdf/gazebo_d400.xacro"/>
             <xacro:gazebo_d400 camera_name="${name}" reference_link="${name}_link" topics_ns="${topics_ns}"
                                depth_optical_frame="${name}_depth_optical_frame"
@@ -119,5 +118,5 @@
                                infrared1_optical_frame="${name}_left_ir_optical_frame"
                                infrared2_optical_frame="${name}_right_ir_optical_frame"
-                               publish_pointcloud="${publish_pointcloud}"/>
+                               publish_pointcloud="${publish_pointcloud}"/> -->
         </xacro:if>
     </xacro:macro>

Commit message: adjusted depth camera pos and made it slower

File: legged_perceptive_description/urdf/robot.xacro (robot description, xacro)
@@ -8,5 +8,5 @@
     <xacro:include filename="$(find legged_perceptive_description)/urdf/nuc_and_lidar/nuc_and_lidar.xacro"/>
     <xacro:sensor_d435 name="front_camera" topics_ns="front_camera" parent="base" sim="true">
-           <origin xyz="0.33 -0.0 0.09" rpy="0 0.83 0"/>
+           <origin xyz="0.2844 -0.0 0.09" rpy="0 0.83 0"/>
       </xacro:sensor_d435>
     <!-- <xacro:sensor_t265 name="tracking_camera" topics_ns="tracking_camera" parent="base">

Commit message: camera orientation stuff

File: legged_perceptive_description/urdf/robot.xacro (robot description, xacro)
@@ -8,5 +8,5 @@
     <xacro:include filename="$(find legged_perceptive_description)/urdf/nuc_and_lidar/nuc_and_lidar.xacro"/>
     <xacro:sensor_d435 name="front_camera" topics_ns="front_camera" parent="base" sim="true">
-           <origin xyz="0.33 -0.0 0.09" rpy="0 0.83 0"/>
+           <origin xyz="0.284 -0.0 0.075" rpy="0 0.87 0"/>
       </xacro:sensor_d435>
     <!-- <xacro:sensor_t265 name="tracking_camera" topics_ns="tracking_camera" parent="base">

Commit message: change cropbox filter dimensions

File: legged_perceptive_description/urdf/robot.xacro (robot description, xacro)
@@ -9,5 +9,4 @@
     <xacro:sensor_d435 name="front_camera" topics_ns="front_camera" parent="base" sim="true">
            <origin xyz="0.284 -0.0 0.075" rpy="0 0.87 0"/>
-           <origin xyz="0.2844 -0.0 0.09" rpy="0 0.83 0"/>
       </xacro:sensor_d435>
     <!-- <xacro:sensor_t265 name="tracking_camera" topics_ns="tracking_camera" parent="base">

Commit message: body filter joystick stuff

File: legged_perceptive_description/urdf/robot.xacro (robot description, xacro)
@@ -8,5 +8,5 @@
     <xacro:include filename="$(find legged_perceptive_description)/urdf/nuc_and_lidar/nuc_and_lidar.xacro"/>
     <xacro:sensor_d435 name="front_camera" topics_ns="front_camera" parent="base" sim="true">
-           <origin xyz="0.284 -0.0 0.075" rpy="0 0.87 0"/>
+           <origin xyz="0.280 -0.0 0.065" rpy="0 0.87 0"/>
       </xacro:sensor_d435>
     <!-- <xacro:sensor_t265 name="tracking_camera" topics_ns="tracking_camera" parent="base">
