Commit message: weight

File: legged_perceptive_description/urdf/nuc_and_lidar/mount.xacro (robot description, xacro)
@@ -2,7 +2,22 @@
     <link name="nuc_top">
         <visual>
-            <origin xyz="0.026999998021894261457 0.045948434504587840066 0.089232763303492723672" rpy="5.509717323009763505e-17 4.2078674255845263165e-14 -3.141592653589793116" />
+            <origin xyz="0.17000000298023223988 0.045999999999999999223 0.038800000000000001155" rpy="0 -0 -1.570796326794896558" />
             <geometry>
-                <mesh filename="$(find legged_perceptive_description)/urdf/nuc_and_lidar/mid-360_lidar_unit.stl"/>
+                <mesh filename="$(find legged_perceptive_description)/urdf/power_holder.stl"/>
+            </geometry>
+            <material name="power_holder_material">
+                <color rgba="0.64705882352941179736 0.64705882352941179736 0.64705882352941179736 1.0"/>
+            </material>
+        </visual>
+        <collision>
+            <origin xyz="0.17000000298023223988 0.045999999999999999223 0.038800000000000001155" rpy="0 -0 -1.570796326794896558" />
+            <geometry>
+                <mesh filename="$(find legged_perceptive_description)/urdf/power_holder.stl"/>
+            </geometry>
+        </collision>
+        <visual>
+            <origin xyz="0.026999998021847469026 0.045828042735641602579 0.081612763303492708022" rpy="6.1232339965243438095e-17 4.2093469295929222686e-14 -3.2595885425187037263e-31" />
+            <geometry>
+                <mesh filename="$(find legged_perceptive_description)/urdf/mid-360_lidar_unit.stl"/>
             </geometry>
             <material name="mid-360_lidar_unit_material">
@@ -11,13 +26,28 @@
         </visual>
         <collision>
-            <origin xyz="0.026999998021894261457 0.045948434504587840066 0.089232763303492723672" rpy="5.509717323009763505e-17 4.2078674255845263165e-14 -3.141592653589793116" />
+            <origin xyz="0.026999998021847469026 0.045828042735641602579 0.081612763303492708022" rpy="6.1232339965243438095e-17 4.2093469295929222686e-14 -3.2595885425187037263e-31" />
             <geometry>
-                <mesh filename="$(find legged_perceptive_description)/urdf/nuc_and_lidar/mid-360_lidar_unit.stl"/>
+                <mesh filename="$(find legged_perceptive_description)/urdf/mid-360_lidar_unit.stl"/>
             </geometry>
         </collision>
         <visual>
-            <origin xyz="0.11750000188499688802 0.092000000234693346535 0.0076199999999999913636" rpy="0 -5.5511151231257827021e-17 3.141592653589793116" />
+            <origin xyz="0.043699998189508933166 0.046000000420958413183 0.054999999999999993339" rpy="3.141592653589793116 -0 -1.570796326794896558" />
             <geometry>
-                <mesh filename="$(find legged_perceptive_description)/urdf/nuc_and_lidar/nuc_enclosure_side.stl"/>
+                <mesh filename="$(find legged_perceptive_description)/urdf/nuc.stl"/>
+            </geometry>
+            <material name="nuc_material">
+                <color rgba="0.4000000000000000222 0.4000000000000000222 0.4000000000000000222 1.0"/>
+            </material>
+        </visual>
+        <collision>
+            <origin xyz="0.043699998189508933166 0.046000000420958413183 0.054999999999999993339" rpy="3.141592653589793116 -0 -1.570796326794896558" />
+            <geometry>
+                <mesh filename="$(find legged_perceptive_description)/urdf/nuc.stl"/>
+            </geometry>
+        </collision>
+        <visual>
+            <origin xyz="0.11750000188499688802 0.092000000234693346535 -3.4694469519536141888e-18" rpy="0 -5.5511151231257827021e-17 3.141592653589793116" />
+            <geometry>
+                <mesh filename="$(find legged_perceptive_description)/urdf/nuc_enclosure_side.stl"/>
             </geometry>
             <material name="nuc_enclosure_side_material">
@@ -26,13 +56,13 @@
         </visual>
         <collision>
-            <origin xyz="0.11750000188499688802 0.092000000234693346535 0.0076199999999999913636" rpy="0 -5.5511151231257827021e-17 3.141592653589793116" />
+            <origin xyz="0.11750000188499688802 0.092000000234693346535 -3.4694469519536141888e-18" rpy="0 -5.5511151231257827021e-17 3.141592653589793116" />
             <geometry>
-                <mesh filename="$(find legged_perceptive_description)/urdf/nuc_and_lidar/nuc_enclosure_side.stl"/>
+                <mesh filename="$(find legged_perceptive_description)/urdf/nuc_enclosure_side.stl"/>
             </geometry>
         </collision>
         <visual>
-            <origin xyz="-0.018000001978128968294 0.017400000130385184088 0.066620000059604680964" rpy="3.141592653589793116 -0 0" />
+            <origin xyz="-0.018000001978128968294 0.017400000130385184088 0.059000000059604665315" rpy="3.141592653589793116 -0 0" />
             <geometry>
-                <mesh filename="$(find legged_perceptive_description)/urdf/nuc_and_lidar/lidar_base.stl"/>
+                <mesh filename="$(find legged_perceptive_description)/urdf/lidar_base.stl"/>
             </geometry>
             <material name="lidar_base_material">
@@ -41,13 +71,13 @@
         </visual>
         <collision>
-            <origin xyz="-0.018000001978128968294 0.017400000130385184088 0.066620000059604680964" rpy="3.141592653589793116 -0 0" />
+            <origin xyz="-0.018000001978128968294 0.017400000130385184088 0.059000000059604665315" rpy="3.141592653589793116 -0 0" />
             <geometry>
-                <mesh filename="$(find legged_perceptive_description)/urdf/nuc_and_lidar/lidar_base.stl"/>
+                <mesh filename="$(find legged_perceptive_description)/urdf/lidar_base.stl"/>
             </geometry>
         </collision>
         <visual>
-            <origin xyz="-0.030500001884996894019 5.5879373633057212225e-11 0.0076200000000000000372" rpy="0 -0 0" />
+            <origin xyz="-0.030500001884996894019 5.5879373633057212225e-11 0" rpy="0 -0 0" />
             <geometry>
-                <mesh filename="$(find legged_perceptive_description)/urdf/nuc_and_lidar/nuc_enclosure_side.stl"/>
+                <mesh filename="$(find legged_perceptive_description)/urdf/nuc_enclosure_side.stl"/>
             </geometry>
             <material name="nuc_enclosure_side_material">
@@ -56,13 +86,13 @@
         </visual>
         <collision>
-            <origin xyz="-0.030500001884996894019 5.5879373633057212225e-11 0.0076200000000000000372" rpy="0 -0 0" />
+            <origin xyz="-0.030500001884996894019 5.5879373633057212225e-11 0" rpy="0 -0 0" />
             <geometry>
-                <mesh filename="$(find legged_perceptive_description)/urdf/nuc_and_lidar/nuc_enclosure_side.stl"/>
+                <mesh filename="$(find legged_perceptive_description)/urdf/nuc_enclosure_side.stl"/>
             </geometry>
         </collision>
         <visual>
-            <origin xyz="0.10975000262260437012 0.10950000036507849532 -1.3919421462405475744e-17" rpy="3.141592653589793116 1.1102230246251565404e-16 0" />
+            <origin xyz="0.10975000262260439787 0.074500000216066925018 -9.039020153071420996e-18" rpy="2.1263491415581675379e-17 1.0678835712080547691e-16 -1.1102230246251562939e-16" />
             <geometry>
-                <mesh filename="$(find legged_perceptive_description)/urdf/nuc_and_lidar/mounting_rail.stl"/>
+                <mesh filename="$(find legged_perceptive_description)/urdf/mounting_rail.stl"/>
             </geometry>
             <material name="mounting_rail_material">
@@ -71,13 +101,13 @@
         </visual>
         <collision>
-            <origin xyz="0.10975000262260437012 0.10950000036507849532 -1.3919421462405475744e-17" rpy="3.141592653589793116 1.1102230246251565404e-16 0" />
+            <origin xyz="0.10975000262260439787 0.074500000216066925018 -9.039020153071420996e-18" rpy="2.1263491415581675379e-17 1.0678835712080547691e-16 -1.1102230246251562939e-16" />
             <geometry>
-                <mesh filename="$(find legged_perceptive_description)/urdf/nuc_and_lidar/mounting_rail.stl"/>
+                <mesh filename="$(find legged_perceptive_description)/urdf/mounting_rail.stl"/>
             </geometry>
         </collision>
         <visual>
-            <origin xyz="-0.018000001978129134828 0.017500000130385186953 0.066620000059604639331" rpy="3.141592653589793116 -0 0" />
+            <origin xyz="-0.018000001978129134828 0.017500000130385186953 0.059000000059604644498" rpy="3.141592653589793116 -0 0" />
             <geometry>
-                <mesh filename="$(find legged_perceptive_description)/urdf/nuc_and_lidar/nuc_top.stl"/>
+                <mesh filename="$(find legged_perceptive_description)/urdf/nuc_top.stl"/>
             </geometry>
             <material name="nuc_top_material">
@@ -86,13 +116,28 @@
         </visual>
         <collision>
-            <origin xyz="-0.018000001978129134828 0.017500000130385186953 0.066620000059604639331" rpy="3.141592653589793116 -0 0" />
+            <origin xyz="-0.018000001978129134828 0.017500000130385186953 0.059000000059604644498" rpy="3.141592653589793116 -0 0" />
             <geometry>
-                <mesh filename="$(find legged_perceptive_description)/urdf/nuc_and_lidar/nuc_top.stl"/>
+                <mesh filename="$(find legged_perceptive_description)/urdf/nuc_top.stl"/>
             </geometry>
         </collision>
         <visual>
-            <origin xyz="0.026999998021870863507 0.045888238620114721322 0.14122000005960458346" rpy="-3.141592653589793116 4.0906603741819780623e-17 -9.9579925010295568285e-17" />
+            <origin xyz="0.071999998021870695308 0.074400000160187468312 0.05910000005960466124" rpy="3.141592653589793116 -0 3.141592653589793116" />
             <geometry>
-                <mesh filename="$(find legged_perceptive_description)/urdf/nuc_and_lidar/frame.stl"/>
+                <mesh filename="$(find legged_perceptive_description)/urdf/lidar_open_guard.stl"/>
+            </geometry>
+            <material name="lidar_open_guard_material">
+                <color rgba="0.61568627450980395466 0.81176470588235294379 0.92941176470588238168 1.0"/>
+            </material>
+        </visual>
+        <collision>
+            <origin xyz="0.071999998021870695308 0.074400000160187468312 0.05910000005960466124" rpy="3.141592653589793116 -0 3.141592653589793116" />
+            <geometry>
+                <mesh filename="$(find legged_perceptive_description)/urdf/lidar_open_guard.stl"/>
+            </geometry>
+        </collision>
+        <visual>
+            <origin xyz="0.026999998021870863507 0.0458882386201147352 0.13360000005960459557" rpy="-3.141592653589793116 2.4370900068556357821e-17 3.141592653589793116" />
+            <geometry>
+                <mesh filename="$(find legged_perceptive_description)/urdf/frame.stl"/>
             </geometry>
             <material name="frame_material">
@@ -101,13 +146,13 @@
         </visual>
         <collision>
-            <origin xyz="0.026999998021870863507 0.045888238620114721322 0.14122000005960458346" rpy="-3.141592653589793116 4.0906603741819780623e-17 -9.9579925010295568285e-17" />
+            <origin xyz="0.026999998021870863507 0.0458882386201147352 0.13360000005960459557" rpy="-3.141592653589793116 2.4370900068556357821e-17 3.141592653589793116" />
             <geometry>
-                <mesh filename="$(find legged_perceptive_description)/urdf/nuc_and_lidar/frame.stl"/>
+                <mesh filename="$(find legged_perceptive_description)/urdf/frame.stl"/>
             </geometry>
         </collision>
         <visual>
-            <origin xyz="0.10975000262260437012 0.017500000074505805969 0" rpy="3.141592653589793116 -0 0" />
+            <origin xyz="0.10975000262260437012 -0.017500000074505805969 0" rpy="0 -0 0" />
             <geometry>
-                <mesh filename="$(find legged_perceptive_description)/urdf/nuc_and_lidar/mounting_rail.stl"/>
+                <mesh filename="$(find legged_perceptive_description)/urdf/mounting_rail.stl"/>
             </geometry>
             <material name="mounting_rail_material">
@@ -116,13 +161,13 @@
         </visual>
         <collision>
-            <origin xyz="0.10975000262260437012 0.017500000074505805969 0" rpy="3.141592653589793116 -0 0" />
+            <origin xyz="0.10975000262260437012 -0.017500000074505805969 0" rpy="0 -0 0" />
             <geometry>
-                <mesh filename="$(find legged_perceptive_description)/urdf/nuc_and_lidar/mounting_rail.stl"/>
+                <mesh filename="$(find legged_perceptive_description)/urdf/mounting_rail.stl"/>
             </geometry>
         </collision>
         <inertial>
-            <origin xyz="0.026999998542501377902 0.046932583314624368165 0.076119999605920501962" rpy="0 0 0"/>
-            <mass value="0.0023640589984545170264" />
-            <inertia ixx="1.7340911567852628544e-07" ixy="1.1255621588591829816e-14" ixz="-1.6675926952365447287e-15" iyy="5.6651910465068455143e-09" iyz="-3.4029341358220793481e-15" izz="1.7366137762786621632e-07" />
+            <origin xyz="0.041012235722627250756 0.045973047634700912878 0.041523664098472856665" rpy="0 0 0"/>
+            <mass value="1.6268089630197246631" />
+            <inertia ixx="0.0031651869174057333661" ixy="-6.1654230755559632426e-07" ixz="0.00027015967922996953713" iyy="0.0031068805832771741876" iyz="2.7450625644812607493e-06" izz="0.0031383494429039287231" />
         </inertial>
     </link>
