Commit message: updated file paths for urdf

File: legged_perceptive_description/urdf/nuc_and_lidar/mount.xacro (robot description, xacro)
@@ -4,5 +4,5 @@
             <origin xyz="0.17000000298023223988 0.045999999999999999223 0.038800000000000001155" rpy="0 -0 -1.570796326794896558" />
             <geometry>
-                <mesh filename="$(find legged_perceptive_description)/urdf/power_holder.stl"/>
+                <mesh filename="$(find legged_perceptive_description)/urdf/nuc_and_lidar/power_holder.stl"/>
             </geometry>
             <material name="power_holder_material">
@@ -13,5 +13,5 @@
             <origin xyz="0.17000000298023223988 0.045999999999999999223 0.038800000000000001155" rpy="0 -0 -1.570796326794896558" />
             <geometry>
-                <mesh filename="$(find legged_perceptive_description)/urdf/power_holder.stl"/>
+                <mesh filename="$(find legged_perceptive_description)/urdf/nuc_and_lidar/power_holder.stl"/>
             </geometry>
         </collision>
@@ -19,5 +19,5 @@
             <origin xyz="0.026999998021847469026 0.045828042735641602579 0.081612763303492708022" rpy="6.1232339965243438095e-17 4.2093469295929222686e-14 -3.2595885425187037263e-31" />
             <geometry>
-                <mesh filename="$(find legged_perceptive_description)/urdf/mid-360_lidar_unit.stl"/>
+                <mesh filename="$(find legged_perceptive_description)/urdf/nuc_and_lidar/mid-360_lidar_unit.stl"/>
             </geometry>
             <material name="mid-360_lidar_unit_material">
@@ -28,5 +28,5 @@
             <origin xyz="0.026999998021847469026 0.045828042735641602579 0.081612763303492708022" rpy="6.1232339965243438095e-17 4.2093469295929222686e-14 -3.2595885425187037263e-31" />
             <geometry>
-                <mesh filename="$(find legged_perceptive_description)/urdf/mid-360_lidar_unit.stl"/>
+                <mesh filename="$(find legged_perceptive_description)/urdf/nuc_and_lidar/mid-360_lidar_unit.stl"/>
             </geometry>
         </collision>
@@ -34,5 +34,5 @@
             <origin xyz="0.043699998189508933166 0.046000000420958413183 0.054999999999999993339" rpy="3.141592653589793116 -0 -1.570796326794896558" />
             <geometry>
-                <mesh filename="$(find legged_perceptive_description)/urdf/nuc.stl"/>
+                <mesh filename="$(find legged_perceptive_description)/urdf/nuc_and_lidar/nuc.stl"/>
             </geometry>
             <material name="nuc_material">
@@ -43,5 +43,5 @@
             <origin xyz="0.043699998189508933166 0.046000000420958413183 0.054999999999999993339" rpy="3.141592653589793116 -0 -1.570796326794896558" />
             <geometry>
-                <mesh filename="$(find legged_perceptive_description)/urdf/nuc.stl"/>
+                <mesh filename="$(find legged_perceptive_description)/urdf/nuc_and_lidar/nuc.stl"/>
             </geometry>
         </collision>
@@ -49,5 +49,5 @@
             <origin xyz="0.11750000188499688802 0.092000000234693346535 -3.4694469519536141888e-18" rpy="0 -5.5511151231257827021e-17 3.141592653589793116" />
             <geometry>
-                <mesh filename="$(find legged_perceptive_description)/urdf/nuc_enclosure_side.stl"/>
+                <mesh filename="$(find legged_perceptive_description)/urdf/nuc_and_lidar/nuc_enclosure_side.stl"/>
             </geometry>
             <material name="nuc_enclosure_side_material">
@@ -58,5 +58,5 @@
             <origin xyz="0.11750000188499688802 0.092000000234693346535 -3.4694469519536141888e-18" rpy="0 -5.5511151231257827021e-17 3.141592653589793116" />
             <geometry>
-                <mesh filename="$(find legged_perceptive_description)/urdf/nuc_enclosure_side.stl"/>
+                <mesh filename="$(find legged_perceptive_description)/urdf/nuc_and_lidar/nuc_enclosure_side.stl"/>
             </geometry>
         </collision>
@@ -64,5 +64,5 @@
             <origin xyz="-0.018000001978128968294 0.017400000130385184088 0.059000000059604665315" rpy="3.141592653589793116 -0 0" />
             <geometry>
-                <mesh filename="$(find legged_perceptive_description)/urdf/lidar_base.stl"/>
+                <mesh filename="$(find legged_perceptive_description)/urdf/nuc_and_lidar/lidar_base.stl"/>
             </geometry>
             <material name="lidar_base_material">
@@ -73,5 +73,5 @@
             <origin xyz="-0.018000001978128968294 0.017400000130385184088 0.059000000059604665315" rpy="3.141592653589793116 -0 0" />
             <geometry>
-                <mesh filename="$(find legged_perceptive_description)/urdf/lidar_base.stl"/>
+                <mesh filename="$(find legged_perceptive_description)/urdf/nuc_and_lidar/lidar_base.stl"/>
             </geometry>
         </collision>
@@ -79,5 +79,5 @@
             <origin xyz="-0.030500001884996894019 5.5879373633057212225e-11 0" rpy="0 -0 0" />
             <geometry>
-                <mesh filename="$(find legged_perceptive_description)/urdf/nuc_enclosure_side.stl"/>
+                <mesh filename="$(find legged_perceptive_description)/urdf/nuc_and_lidar/nuc_enclosure_side.stl"/>
             </geometry>
             <material name="nuc_enclosure_side_material">
@@ -88,5 +88,5 @@
             <origin xyz="-0.030500001884996894019 5.5879373633057212225e-11 0" rpy="0 -0 0" />
             <geometry>
-                <mesh filename="$(find legged_perceptive_description)/urdf/nuc_enclosure_side.stl"/>
+                <mesh filename="$(find legged_perceptive_description)/urdf/nuc_and_lidar/nuc_enclosure_side.stl"/>
             </geometry>
         </collision>
@@ -94,5 +94,5 @@
             <origin xyz="0.10975000262260439787 0.074500000216066925018 -9.039020153071420996e-18" rpy="2.1263491415581675379e-17 1.0678835712080547691e-16 -1.1102230246251562939e-16" />
             <geometry>
-                <mesh filename="$(find legged_perceptive_description)/urdf/mounting_rail.stl"/>
+                <mesh filename="$(find legged_perceptive_description)/urdf/nuc_and_lidar/mounting_rail.stl"/>
             </geometry>
             <material name="mounting_rail_material">
@@ -103,5 +103,5 @@
             <origin xyz="0.10975000262260439787 0.074500000216066925018 -9.039020153071420996e-18" rpy="2.1263491415581675379e-17 1.0678835712080547691e-16 -1.1102230246251562939e-16" />
             <geometry>
-                <mesh filename="$(find legged_perceptive_description)/urdf/mounting_rail.stl"/>
+                <mesh filename="$(find legged_perceptive_description)/urdf/nuc_and_lidar/mounting_rail.stl"/>
             </geometry>
         </collision>
@@ -109,5 +109,5 @@
             <origin xyz="-0.018000001978129134828 0.017500000130385186953 0.059000000059604644498" rpy="3.141592653589793116 -0 0" />
             <geometry>
-                <mesh filename="$(find legged_perceptive_description)/urdf/nuc_top.stl"/>
+                <mesh filename="$(find legged_perceptive_description)/urdf/nuc_and_lidar/nuc_top.stl"/>
             </geometry>
             <material name="nuc_top_material">
@@ -118,5 +118,5 @@
             <origin xyz="-0.018000001978129134828 0.017500000130385186953 0.059000000059604644498" rpy="3.141592653589793116 -0 0" />
             <geometry>
-                <mesh filename="$(find legged_perceptive_description)/urdf/nuc_top.stl"/>
+                <mesh filename="$(find legged_perceptive_description)/urdf/nuc_and_lidar/nuc_top.stl"/>
             </geometry>
         </collision>
@@ -124,5 +124,5 @@
             <origin xyz="0.071999998021870695308 0.074400000160187468312 0.05910000005960466124" rpy="3.141592653589793116 -0 3.141592653589793116" />
             <geometry>
-                <mesh filename="$(find legged_perceptive_description)/urdf/lidar_open_guard.stl"/>
+                <mesh filename="$(find legged_perceptive_description)/urdf/nuc_and_lidar/lidar_open_guard.stl"/>
             </geometry>
             <material name="lidar_open_guard_material">
@@ -133,5 +133,5 @@
             <origin xyz="0.071999998021870695308 0.074400000160187468312 0.05910000005960466124" rpy="3.141592653589793116 -0 3.141592653589793116" />
             <geometry>
-                <mesh filename="$(find legged_perceptive_description)/urdf/lidar_open_guard.stl"/>
+                <mesh filename="$(find legged_perceptive_description)/urdf/nuc_and_lidar/lidar_open_guard.stl"/>
             </geometry>
         </collision>
@@ -139,5 +139,5 @@
             <origin xyz="0.026999998021870863507 0.0458882386201147352 0.13360000005960459557" rpy="-3.141592653589793116 2.4370900068556357821e-17 3.141592653589793116" />
             <geometry>
-                <mesh filename="$(find legged_perceptive_description)/urdf/frame.stl"/>
+                <mesh filename="$(find legged_perceptive_description)/urdf/nuc_and_lidar/frame.stl"/>
             </geometry>
             <material name="frame_material">
@@ -148,5 +148,5 @@
             <origin xyz="0.026999998021870863507 0.0458882386201147352 0.13360000005960459557" rpy="-3.141592653589793116 2.4370900068556357821e-17 3.141592653589793116" />
             <geometry>
-                <mesh filename="$(find legged_perceptive_description)/urdf/frame.stl"/>
+                <mesh filename="$(find legged_perceptive_description)/urdf/nuc_and_lidar/frame.stl"/>
             </geometry>
         </collision>
@@ -154,5 +154,5 @@
             <origin xyz="0.10975000262260437012 -0.017500000074505805969 0" rpy="0 -0 0" />
             <geometry>
-                <mesh filename="$(find legged_perceptive_description)/urdf/mounting_rail.stl"/>
+                <mesh filename="$(find legged_perceptive_description)/urdf/nuc_and_lidar/mounting_rail.stl"/>
             </geometry>
             <material name="mounting_rail_material">
@@ -163,5 +163,5 @@
             <origin xyz="0.10975000262260437012 -0.017500000074505805969 0" rpy="0 -0 0" />
             <geometry>
-                <mesh filename="$(find legged_perceptive_description)/urdf/mounting_rail.stl"/>
+                <mesh filename="$(find legged_perceptive_description)/urdf/nuc_and_lidar/mounting_rail.stl"/>
             </geometry>
         </collision>

Commit message: elevation mapping using lidar on robot

File: legged_perceptive_description/urdf/nuc_and_lidar/mount.xacro (robot description, xacro)
@@ -4,5 +4,5 @@
             <origin xyz="0.17000000298023223988 0.045999999999999999223 0.038800000000000001155" rpy="0 -0 -1.570796326794896558" />
             <geometry>
-                <mesh filename="$(find legged_perceptive_description)/urdf/nuc_and_lidar/power_holder.stl"/>
+                <mesh filename="file://$(find legged_perceptive_description)/urdf/nuc_and_lidar/power_holder.stl"/>
             </geometry>
             <material name="power_holder_material">
@@ -13,5 +13,5 @@
             <origin xyz="0.17000000298023223988 0.045999999999999999223 0.038800000000000001155" rpy="0 -0 -1.570796326794896558" />
             <geometry>
-                <mesh filename="$(find legged_perceptive_description)/urdf/nuc_and_lidar/power_holder.stl"/>
+                <mesh filename="file://$(find legged_perceptive_description)/urdf/nuc_and_lidar/power_holder.stl"/>
             </geometry>
         </collision>
@@ -19,5 +19,5 @@
             <origin xyz="0.026999998021847469026 0.045828042735641602579 0.081612763303492708022" rpy="6.1232339965243438095e-17 4.2093469295929222686e-14 -3.2595885425187037263e-31" />
             <geometry>
-                <mesh filename="$(find legged_perceptive_description)/urdf/nuc_and_lidar/mid-360_lidar_unit.stl"/>
+                <mesh filename="file://$(find legged_perceptive_description)/urdf/nuc_and_lidar/mid-360_lidar_unit.stl"/>
             </geometry>
             <material name="mid-360_lidar_unit_material">
@@ -28,5 +28,5 @@
             <origin xyz="0.026999998021847469026 0.045828042735641602579 0.081612763303492708022" rpy="6.1232339965243438095e-17 4.2093469295929222686e-14 -3.2595885425187037263e-31" />
             <geometry>
-                <mesh filename="$(find legged_perceptive_description)/urdf/nuc_and_lidar/mid-360_lidar_unit.stl"/>
+                <mesh filename="file://$(find legged_perceptive_description)/urdf/nuc_and_lidar/mid-360_lidar_unit.stl"/>
             </geometry>
         </collision>
@@ -34,5 +34,5 @@
             <origin xyz="0.043699998189508933166 0.046000000420958413183 0.054999999999999993339" rpy="3.141592653589793116 -0 -1.570796326794896558" />
             <geometry>
-                <mesh filename="$(find legged_perceptive_description)/urdf/nuc_and_lidar/nuc.stl"/>
+                <mesh filename="file://$(find legged_perceptive_description)/urdf/nuc_and_lidar/nuc.stl"/>
             </geometry>
             <material name="nuc_material">
@@ -43,5 +43,5 @@
             <origin xyz="0.043699998189508933166 0.046000000420958413183 0.054999999999999993339" rpy="3.141592653589793116 -0 -1.570796326794896558" />
             <geometry>
-                <mesh filename="$(find legged_perceptive_description)/urdf/nuc_and_lidar/nuc.stl"/>
+                <mesh filename="file://$(find legged_perceptive_description)/urdf/nuc_and_lidar/nuc.stl"/>
             </geometry>
         </collision>
@@ -49,5 +49,5 @@
             <origin xyz="0.11750000188499688802 0.092000000234693346535 -3.4694469519536141888e-18" rpy="0 -5.5511151231257827021e-17 3.141592653589793116" />
             <geometry>
-                <mesh filename="$(find legged_perceptive_description)/urdf/nuc_and_lidar/nuc_enclosure_side.stl"/>
+                <mesh filename="file://$(find legged_perceptive_description)/urdf/nuc_and_lidar/nuc_enclosure_side.stl"/>
             </geometry>
             <material name="nuc_enclosure_side_material">
@@ -58,5 +58,5 @@
             <origin xyz="0.11750000188499688802 0.092000000234693346535 -3.4694469519536141888e-18" rpy="0 -5.5511151231257827021e-17 3.141592653589793116" />
             <geometry>
-                <mesh filename="$(find legged_perceptive_description)/urdf/nuc_and_lidar/nuc_enclosure_side.stl"/>
+                <mesh filename="file://$(find legged_perceptive_description)/urdf/nuc_and_lidar/nuc_enclosure_side.stl"/>
             </geometry>
         </collision>
@@ -64,5 +64,5 @@
             <origin xyz="-0.018000001978128968294 0.017400000130385184088 0.059000000059604665315" rpy="3.141592653589793116 -0 0" />
             <geometry>
-                <mesh filename="$(find legged_perceptive_description)/urdf/nuc_and_lidar/lidar_base.stl"/>
+                <mesh filename="file://$(find legged_perceptive_description)/urdf/nuc_and_lidar/lidar_base.stl"/>
             </geometry>
             <material name="lidar_base_material">
@@ -73,5 +73,5 @@
             <origin xyz="-0.018000001978128968294 0.017400000130385184088 0.059000000059604665315" rpy="3.141592653589793116 -0 0" />
             <geometry>
-                <mesh filename="$(find legged_perceptive_description)/urdf/nuc_and_lidar/lidar_base.stl"/>
+                <mesh filename="file://$(find legged_perceptive_description)/urdf/nuc_and_lidar/lidar_base.stl"/>
             </geometry>
         </collision>
@@ -79,5 +79,5 @@
             <origin xyz="-0.030500001884996894019 5.5879373633057212225e-11 0" rpy="0 -0 0" />
             <geometry>
-                <mesh filename="$(find legged_perceptive_description)/urdf/nuc_and_lidar/nuc_enclosure_side.stl"/>
+                <mesh filename="file://$(find legged_perceptive_description)/urdf/nuc_and_lidar/nuc_enclosure_side.stl"/>
             </geometry>
             <material name="nuc_enclosure_side_material">
@@ -88,5 +88,5 @@
             <origin xyz="-0.030500001884996894019 5.5879373633057212225e-11 0" rpy="0 -0 0" />
             <geometry>
-                <mesh filename="$(find legged_perceptive_description)/urdf/nuc_and_lidar/nuc_enclosure_side.stl"/>
+                <mesh filename="file://$(find legged_perceptive_description)/urdf/nuc_and_lidar/nuc_enclosure_side.stl"/>
             </geometry>
         </collision>
@@ -94,5 +94,5 @@
             <origin xyz="0.10975000262260439787 0.074500000216066925018 -9.039020153071420996e-18" rpy="2.1263491415581675379e-17 1.0678835712080547691e-16 -1.1102230246251562939e-16" />
             <geometry>
-                <mesh filename="$(find legged_perceptive_description)/urdf/nuc_and_lidar/mounting_rail.stl"/>
+                <mesh filename="file://$(find legged_perceptive_description)/urdf/nuc_and_lidar/mounting_rail.stl"/>
             </geometry>
             <material name="mounting_rail_material">
@@ -103,5 +103,5 @@
             <origin xyz="0.10975000262260439787 0.074500000216066925018 -9.039020153071420996e-18" rpy="2.1263491415581675379e-17 1.0678835712080547691e-16 -1.1102230246251562939e-16" />
             <geometry>
-                <mesh filename="$(find legged_perceptive_description)/urdf/nuc_and_lidar/mounting_rail.stl"/>
+                <mesh filename="file://$(find legged_perceptive_description)/urdf/nuc_and_lidar/mounting_rail.stl"/>
             </geometry>
         </collision>
@@ -109,5 +109,5 @@
             <origin xyz="-0.018000001978129134828 0.017500000130385186953 0.059000000059604644498" rpy="3.141592653589793116 -0 0" />
             <geometry>
-                <mesh filename="$(find legged_perceptive_description)/urdf/nuc_and_lidar/nuc_top.stl"/>
+                <mesh filename="file://$(find legged_perceptive_description)/urdf/nuc_and_lidar/nuc_top.stl"/>
             </geometry>
             <material name="nuc_top_material">
@@ -118,5 +118,5 @@
             <origin xyz="-0.018000001978129134828 0.017500000130385186953 0.059000000059604644498" rpy="3.141592653589793116 -0 0" />
             <geometry>
-                <mesh filename="$(find legged_perceptive_description)/urdf/nuc_and_lidar/nuc_top.stl"/>
+                <mesh filename="file://$(find legged_perceptive_description)/urdf/nuc_and_lidar/nuc_top.stl"/>
             </geometry>
         </collision>
@@ -124,5 +124,5 @@
             <origin xyz="0.071999998021870695308 0.074400000160187468312 0.05910000005960466124" rpy="3.141592653589793116 -0 3.141592653589793116" />
             <geometry>
-                <mesh filename="$(find legged_perceptive_description)/urdf/nuc_and_lidar/lidar_open_guard.stl"/>
+                <mesh filename="file://$(find legged_perceptive_description)/urdf/nuc_and_lidar/lidar_open_guard.stl"/>
             </geometry>
             <material name="lidar_open_guard_material">
@@ -133,5 +133,5 @@
             <origin xyz="0.071999998021870695308 0.074400000160187468312 0.05910000005960466124" rpy="3.141592653589793116 -0 3.141592653589793116" />
             <geometry>
-                <mesh filename="$(find legged_perceptive_description)/urdf/nuc_and_lidar/lidar_open_guard.stl"/>
+                <mesh filename="file://$(find legged_perceptive_description)/urdf/nuc_and_lidar/lidar_open_guard.stl"/>
             </geometry>
         </collision>
@@ -139,5 +139,5 @@
             <origin xyz="0.026999998021870863507 0.0458882386201147352 0.13360000005960459557" rpy="-3.141592653589793116 2.4370900068556357821e-17 3.141592653589793116" />
             <geometry>
-                <mesh filename="$(find legged_perceptive_description)/urdf/nuc_and_lidar/frame.stl"/>
+                <mesh filename="file://$(find legged_perceptive_description)/urdf/nuc_and_lidar/frame.stl"/>
             </geometry>
             <material name="frame_material">
@@ -148,5 +148,5 @@
             <origin xyz="0.026999998021870863507 0.0458882386201147352 0.13360000005960459557" rpy="-3.141592653589793116 2.4370900068556357821e-17 3.141592653589793116" />
             <geometry>
-                <mesh filename="$(find legged_perceptive_description)/urdf/nuc_and_lidar/frame.stl"/>
+                <mesh filename="file://$(find legged_perceptive_description)/urdf/nuc_and_lidar/frame.stl"/>
             </geometry>
         </collision>
@@ -154,5 +154,5 @@
             <origin xyz="0.10975000262260437012 -0.017500000074505805969 0" rpy="0 -0 0" />
             <geometry>
-                <mesh filename="$(find legged_perceptive_description)/urdf/nuc_and_lidar/mounting_rail.stl"/>
+                <mesh filename="file://$(find legged_perceptive_description)/urdf/nuc_and_lidar/mounting_rail.stl"/>
             </geometry>
             <material name="mounting_rail_material">
@@ -163,5 +163,5 @@
             <origin xyz="0.10975000262260437012 -0.017500000074505805969 0" rpy="0 -0 0" />
             <geometry>
-                <mesh filename="$(find legged_perceptive_description)/urdf/nuc_and_lidar/mounting_rail.stl"/>
+                <mesh filename="file://$(find legged_perceptive_description)/urdf/nuc_and_lidar/mounting_rail.stl"/>
             </geometry>
         </collision>

File: legged_perceptive_description/urdf/robot.xacro (robot description, xacro)
@@ -20,3 +20,8 @@
         <origin xyz="0.365 0.068 -0.030" rpy="2.59 1.03 -3.09"/>
     </xacro:Livox_Mid360> -->
+    <!-- <joint name="camera_init_joint" type="fixed">
+        <parent link="lidar_frame"/>
+        <child link="camera_init"/>
+        <origin xyz="0 0 0" rpy="0 0 0"/>
+    </joint> -->
 </robot>
