Commit message: fixed urdf

File: legged_perceptive_description/urdf/nuc_and_lidar/nuc_and_lidar.xacro (robot description, xacro)
@@ -14,5 +14,5 @@
         <parent link="base"/>
         <child link="nuc_top"/>
-        <origin xyz="0.0 0.0 0.7" rpy="3.141592653589793116 0 0"/>
+        <origin xyz="0.10975 0.046 0.0575" rpy="3.141592653589793116 3.141592653589793116 0"/>
     </joint>
 </robot>

Commit message: slam working ??

File: legged_perceptive_description/urdf/nuc_and_lidar/nuc_and_lidar.xacro (robot description, xacro)
@@ -10,4 +10,12 @@
         <origin xyz="0.026999998021870863507 0.045888238620114721322 0.13622000005960458346" rpy="-3.141592653589793116 -3.141592653589793116 -9.9579925010295568285e-17"/>
     </joint>
+    <link name="lidar_imu_frame"/>
+    <!-- Fixed Joint to attach lidar_imu_frame to lidar_frame using the provided extrinsics -->
+    <joint name="lidar_imu_joint" type="fixed">
+    <parent link="lidar_frame"/>
+    <child link="lidar_imu_frame"/>
+    <!-- Extrinsics: translation from lidar_frame and identity rotation -->
+    <origin xyz="0.011 0.02329 -0.04412" rpy="0 0 0"/>
+    </joint>
     <!-- Joint to attach nuc_top to base -->
     <joint name="nuc_top_joint" type="fixed">

Commit message: slam

File: legged_perceptive_description/urdf/nuc_and_lidar/nuc_and_lidar.xacro (robot description, xacro)
@@ -16,5 +16,5 @@
     <child link="lidar_imu_frame"/>
     <!-- Extrinsics: translation from lidar_frame and identity rotation -->
-    <origin xyz="0.011 0.02329 -0.04412" rpy="0 0 0"/>
+    <origin xyz="-0.011 -0.02329 0.04412" rpy="0 0 0"/>
     </joint>
     <!-- Joint to attach nuc_top to base -->

Commit message: updated NUC and Lidar mount xacro

File: legged_perceptive_description/urdf/nuc_and_lidar/nuc_and_lidar.xacro (robot description, xacro)
@@ -2,5 +2,5 @@
 <robot xmlns:xacro="http://www.ros.org/wiki/xacro" name="onshape_with_lidar">
     <!-- Import the main URDF file -->
-    <xacro:include filename="mount.xacro"/>
+    <xacro:include filename="mount_2.xacro"/>
     <link name="lidar_frame"/>
     <!-- Fixed Joint to Attach lidar_frame to nuc_top -->
@@ -22,5 +22,5 @@
         <parent link="base"/>
         <child link="nuc_top"/>
-        <origin xyz="0.10975 0.046 0.0575" rpy="3.141592653589793116 3.141592653589793116 0"/>
+        <origin xyz="0.10975 0.046 0.0648" rpy="3.141592653589793116 3.141592653589793116 0"/>
     </joint>
 </robot>

Commit message: lidar changes and elevation map param changes

File: legged_perceptive_description/urdf/nuc_and_lidar/nuc_and_lidar.xacro (robot description, xacro)
@@ -16,5 +16,5 @@
     <child link="lidar_imu_frame"/>
     <!-- Extrinsics: translation from lidar_frame and identity rotation -->
-    <origin xyz="-0.011 -0.02329 0.04412" rpy="0 0 0"/>
+    <origin xyz="0.011 0.02329 -0.04412" rpy="0 0 0"/>
     </joint>
     <!-- Joint to attach nuc_top to base -->
