Commit message: updated weights and made 3rd mount xacro

File: legged_perceptive_description/urdf/nuc_and_lidar/mount_3.xacro (robot description, xacro)
@@ -1,7 +1,5 @@
-<?xml version="1.0" ?>
+<robot xmlns:xacro="http://www.ros.org/wiki/xacro" name="onshape">
 <!-- Generated using onshape-to-robot -->
-<robot name="onshape">
-    <!-- Link mid-360_lidar_unit -->
-    <link name="mid-360_lidar_unit">
+    <link name="nuc_top">
         <inertial>
             <origin xyz="0.0900752 0.04556 0.0470702" rpy="0 0 0"/>
@@ -13,5 +11,5 @@
             <origin xyz="-0.018 0.0175 0.059" rpy="3.14159 -0 0"/>
             <geometry>
-                <mesh filename="package://legged_perceptive_description/urdf/nuc_and_lidar/nuc_top.stl"/>
+                <mesh filename="file://$(find legged_perceptive_description)/urdf/nuc_and_lidar/nuc_top.stl"/>
             </geometry>
             <material name="nuc_top_material">
@@ -22,5 +20,5 @@
             <origin xyz="-0.018 0.0175 0.059" rpy="3.14159 -0 0"/>
             <geometry>
-                <mesh filename="package://legged_perceptive_description/urdf/nuc_and_lidar/nuc_top.stl"/>
+                <mesh filename="file://$(find legged_perceptive_description)/urdf/nuc_and_lidar/nuc_top.stl"/>
             </geometry>
         </collision>
@@ -29,5 +27,5 @@
             <origin xyz="0.027 0.0460004 0.0816128" rpy="6.12323e-17 4.20935e-14 -1.71018e-46"/>
             <geometry>
-                <mesh filename="package://legged_perceptive_description/urdf/nuc_and_lidar/mid_360_lidar_unit.stl"/>
+                <mesh filename="file://$(find legged_perceptive_description)/urdf/nuc_and_lidar/mid_360_lidar_unit.stl"/>
             </geometry>
             <material name="mid-360_lidar_unit_material">
@@ -38,5 +36,5 @@
             <origin xyz="0.027 0.0460004 0.0816128" rpy="6.12323e-17 4.20935e-14 -1.71018e-46"/>
             <geometry>
-                <mesh filename="package://legged_perceptive_description/urdf/nuc_and_lidar/mid_360_lidar_unit.stl"/>
+                <mesh filename="file://$(find legged_perceptive_description)/urdf/nuc_and_lidar/mid_360_lidar_unit.stl"/>
             </geometry>
         </collision>
@@ -45,5 +43,5 @@
             <origin xyz="0.1705 0.046 0.049" rpy="1.01161e-46 -2.30521e-16 -3.14159"/>
             <geometry>
-                <mesh filename="package://legged_perceptive_description/urdf/nuc_and_lidar/voltageregulatormount.stl"/>
+                <mesh filename="file://$(find legged_perceptive_description)/urdf/nuc_and_lidar/voltageregulatormount.stl"/>
             </geometry>
             <material name="voltageregulatormount_material">
@@ -54,5 +52,5 @@
             <origin xyz="0.1705 0.046 0.049" rpy="1.01161e-46 -2.30521e-16 -3.14159"/>
             <geometry>
-                <mesh filename="package://legged_perceptive_description/urdf/nuc_and_lidar/voltageregulatormount.stl"/>
+                <mesh filename="file://$(find legged_perceptive_description)/urdf/nuc_and_lidar/voltageregulatormount.stl"/>
             </geometry>
         </collision>
@@ -61,5 +59,5 @@
             <origin xyz="0.044 0.046 0.05" rpy="3.14159 -0 -1.5708"/>
             <geometry>
-                <mesh filename="package://legged_perceptive_description/urdf/nuc_and_lidar/nuc.stl"/>
+                <mesh filename="file://$(find legged_perceptive_description)/urdf/nuc_and_lidar/nuc.stl"/>
             </geometry>
             <material name="nuc_material">
@@ -70,5 +68,5 @@
             <origin xyz="0.044 0.046 0.05" rpy="3.14159 -0 -1.5708"/>
             <geometry>
-                <mesh filename="package://legged_perceptive_description/urdf/nuc_and_lidar/nuc.stl"/>
+                <mesh filename="file://$(find legged_perceptive_description)/urdf/nuc_and_lidar/nuc.stl"/>
             </geometry>
         </collision>
@@ -77,5 +75,5 @@
             <origin xyz="0.1175 0.092 -2.60209e-18" rpy="0 -0 3.14159"/>
             <geometry>
-                <mesh filename="package://legged_perceptive_description/urdf/nuc_and_lidar/nuc_enclosure_side.stl"/>
+                <mesh filename="file://$(find legged_perceptive_description)/urdf/nuc_and_lidar/nuc_enclosure_side.stl"/>
             </geometry>
             <material name="nuc_enclosure_side_material">
@@ -86,5 +84,5 @@
             <origin xyz="0.1175 0.092 -2.60209e-18" rpy="0 -0 3.14159"/>
             <geometry>
-                <mesh filename="package://legged_perceptive_description/urdf/nuc_and_lidar/nuc_enclosure_side.stl"/>
+                <mesh filename="file://$(find legged_perceptive_description)/urdf/nuc_and_lidar/nuc_enclosure_side.stl"/>
             </geometry>
         </collision>
@@ -93,5 +91,5 @@
             <origin xyz="-0.0305 5.58794e-11 0" rpy="0 -0 0"/>
             <geometry>
-                <mesh filename="package://legged_perceptive_description/urdf/nuc_and_lidar/nuc_enclosure_side.stl"/>
+                <mesh filename="file://$(find legged_perceptive_description)/urdf/nuc_and_lidar/nuc_enclosure_side.stl"/>
             </geometry>
             <material name="nuc_enclosure_side_2_material">
@@ -102,5 +100,5 @@
             <origin xyz="-0.0305 5.58794e-11 0" rpy="0 -0 0"/>
             <geometry>
-                <mesh filename="package://legged_perceptive_description/urdf/nuc_and_lidar/nuc_enclosure_side.stl"/>
+                <mesh filename="file://$(find legged_perceptive_description)/urdf/nuc_and_lidar/nuc_enclosure_side.stl"/>
             </geometry>
         </collision>
@@ -109,5 +107,5 @@
             <origin xyz="0.10975 0.0745 -2.60209e-18" rpy="-6.16298e-33 -1.2326e-32 -2.77556e-17"/>
             <geometry>
-                <mesh filename="package://legged_perceptive_description/urdf/nuc_and_lidar/mounting_rail.stl"/>
+                <mesh filename="file://$(find legged_perceptive_description)/urdf/nuc_and_lidar/mounting_rail.stl"/>
             </geometry>
             <material name="mounting_rail_material">
@@ -118,5 +116,5 @@
             <origin xyz="0.10975 0.0745 -2.60209e-18" rpy="-6.16298e-33 -1.2326e-32 -2.77556e-17"/>
             <geometry>
-                <mesh filename="package://legged_perceptive_description/urdf/nuc_and_lidar/mounting_rail.stl"/>
+                <mesh filename="file://$(find legged_perceptive_description)/urdf/nuc_and_lidar/mounting_rail.stl"/>
             </geometry>
         </collision>
@@ -125,5 +123,5 @@
             <origin xyz="0.169134 0.046 0.063" rpy="-2.30521e-16 -1.01161e-46 -1.5708"/>
             <geometry>
-                <mesh filename="package://legged_perceptive_description/urdf/nuc_and_lidar/psu.stl"/>
+                <mesh filename="file://$(find legged_perceptive_description)/urdf/nuc_and_lidar/psu.stl"/>
             </geometry>
             <material name="psu_material">
@@ -134,5 +132,5 @@
             <origin xyz="0.169134 0.046 0.063" rpy="-2.30521e-16 -1.01161e-46 -1.5708"/>
             <geometry>
-                <mesh filename="package://legged_perceptive_description/urdf/nuc_and_lidar/psu.stl"/>
+                <mesh filename="file://$(find legged_perceptive_description)/urdf/nuc_and_lidar/psu.stl"/>
             </geometry>
         </collision>
@@ -141,5 +139,5 @@
             <origin xyz="0.1725 0.008 0.026" rpy="-1.5708 2.30521e-16 0"/>
             <geometry>
-                <mesh filename="package://legged_perceptive_description/urdf/nuc_and_lidar/battery.stl"/>
+                <mesh filename="file://$(find legged_perceptive_description)/urdf/nuc_and_lidar/battery.stl"/>
             </geometry>
             <material name="battery_material">
@@ -150,5 +148,5 @@
             <origin xyz="0.1725 0.008 0.026" rpy="-1.5708 2.30521e-16 0"/>
             <geometry>
-                <mesh filename="package://legged_perceptive_description/urdf/nuc_and_lidar/battery.stl"/>
+                <mesh filename="file://$(find legged_perceptive_description)/urdf/nuc_and_lidar/battery.stl"/>
             </geometry>
         </collision>
@@ -157,5 +155,5 @@
             <origin xyz="0.027 0.0460605 0.1336" rpy="-3.14159 2.43709e-17 3.14159"/>
             <geometry>
-                <mesh filename="package://legged_perceptive_description/urdf/nuc_and_lidar/frame.stl"/>
+                <mesh filename="file://$(find legged_perceptive_description)/urdf/nuc_and_lidar/frame.stl"/>
             </geometry>
             <material name="frame_material">
@@ -166,5 +164,5 @@
             <origin xyz="0.027 0.0460605 0.1336" rpy="-3.14159 2.43709e-17 3.14159"/>
             <geometry>
-                <mesh filename="package://legged_perceptive_description/urdf/nuc_and_lidar/frame.stl"/>
+                <mesh filename="file://$(find legged_perceptive_description)/urdf/nuc_and_lidar/frame.stl"/>
             </geometry>
         </collision>
@@ -173,5 +171,5 @@
             <origin xyz="0.10975 -0.0175 0" rpy="0 -0 0"/>
             <geometry>
-                <mesh filename="package://legged_perceptive_description/urdf/nuc_and_lidar/mounting_rail.stl"/>
+                <mesh filename="file://$(find legged_perceptive_description)/urdf/nuc_and_lidar/mounting_rail.stl"/>
             </geometry>
             <material name="mounting_rail_2_material">
@@ -182,5 +180,5 @@
             <origin xyz="0.10975 -0.0175 0" rpy="0 -0 0"/>
             <geometry>
-                <mesh filename="package://legged_perceptive_description/urdf/nuc_and_lidar/mounting_rail.stl"/>
+                <mesh filename="file://$(find legged_perceptive_description)/urdf/nuc_and_lidar/mounting_rail.stl"/>
             </geometry>
         </collision>
@@ -189,5 +187,5 @@
             <origin xyz="0.1745 0.046 -6.93889e-18" rpy="-2.30521e-16 -0 -1.5708"/>
             <geometry>
-                <mesh filename="package://legged_perceptive_description/urdf/nuc_and_lidar/batterymount.stl"/>
+                <mesh filename="file://$(find legged_perceptive_description)/urdf/nuc_and_lidar/batterymount.stl"/>
             </geometry>
             <material name="batterymount_material">
@@ -198,5 +196,5 @@
             <origin xyz="0.1745 0.046 -6.93889e-18" rpy="-2.30521e-16 -0 -1.5708"/>
             <geometry>
-                <mesh filename="package://legged_perceptive_description/urdf/nuc_and_lidar/batterymount.stl"/>
+                <mesh filename="file://$(find legged_perceptive_description)/urdf/nuc_and_lidar/batterymount.stl"/>
             </geometry>
         </collision>

File: legged_perceptive_description/urdf/nuc_and_lidar/nuc_and_lidar.xacro (robot description, xacro)
@@ -2,5 +2,5 @@
 <robot xmlns:xacro="http://www.ros.org/wiki/xacro" name="onshape_with_lidar">
     <!-- Import the main URDF file -->
-    <xacro:include filename="mount_2.xacro"/>
+    <xacro:include filename="mount_3.xacro"/>
     <link name="lidar_frame"/>
     <!-- Fixed Joint to Attach lidar_frame to nuc_top -->

Commit message: forgor to comment out the little thing at the end

File: legged_perceptive_description/urdf/nuc_and_lidar/mount_3.xacro (robot description, xacro)
@@ -201,5 +201,5 @@
     </link>
     <!-- Frame livox (dummy link + fixed joint) -->
-    <link name="livox">
+    <!-- <link name="livox">
         <origin xyz="0 0 0" rpy="0 -0 0"/>
         <inertial>
@@ -214,4 +214,4 @@
         <child link="livox"/>
         <axis xyz="0 0 0"/>
-    </joint>
+    </joint> -->
 </robot>
