Commit message: added ne nuc and lidar xacro for the slanted config

File: legged_perceptive_description/urdf/nuc_and_lidar/mount_4.xacro (robot description, xacro)
@@ -1,33 +1,16 @@
-<?xml version="1.0" ?>
+<robot xmlns:xacro="http://www.ros.org/wiki/xacro" name="onshape">
 <!-- Generated using onshape-to-robot -->
-<robot name="onshape">
     <!-- Link mid-360_lidar_unit -->
-    <link name="mid-360_lidar_unit">
+    <link name="nuc_top">
         <inertial>
-            <origin xyz="0.0900752 0.04556 0.0470702" rpy="0 0 0"/>
-            <mass value="1.55055"/>
-            <inertia ixx="0.00269047" ixy="7.5858e-05" ixz="0.000944732" iyy="0.00919912" iyz="-1.44756e-05" izz="0.00855227"/>
+            <origin xyz="0.0919709 0.0455289 0.0500946" rpy="0 0 0"/>
+            <mass value="1.44797"/>
+            <inertia ixx="0.00341863" ixy="7.45764e-05" ixz="0.00146802" iyy="0.00992739" iyz="-1.65902e-05" izz="0.00842917"/>
         </inertial>
-        <!-- Part nuc_top -->
-        <visual>
-            <origin xyz="-0.018 0.0175 0.059" rpy="3.14159 -0 0"/>
-            <geometry>
-                <mesh filename="package://legged_perceptive_description/urdf/nuc_and_lidar/nuc_top.stl"/>
-            </geometry>
-            <material name="nuc_top_material">
-                <color rgba="0.917647 0.917647 0.917647 1.0"/>
-            </material>
-        </visual>
-        <collision>
-            <origin xyz="-0.018 0.0175 0.059" rpy="3.14159 -0 0"/>
-            <geometry>
-                <mesh filename="package://legged_perceptive_description/urdf/nuc_and_lidar/nuc_top.stl"/>
-            </geometry>
-        </collision>
         <!-- Part mid-360_lidar_unit -->
         <visual>
-            <origin xyz="0.027 0.0460004 0.0816128" rpy="6.12323e-17 4.20935e-14 -1.71018e-46"/>
-            <geometry>
-                <mesh filename="package://legged_perceptive_description/urdf/nuc_and_lidar/mid_360_lidar_unit.stl"/>
+            <origin xyz="0.0240064 0.0460004 0.106664" rpy="6.12323e-17 -0.383972 -6.93889e-18"/>
+            <geometry>
+                <mesh filename="file://$(find legged_perceptive_description)/urdf/nuc_and_lidar/mid_360_lidar_unit.stl"/>
             </geometry>
             <material name="mid-360_lidar_unit_material">
@@ -36,7 +19,7 @@
         </visual>
         <collision>
-            <origin xyz="0.027 0.0460004 0.0816128" rpy="6.12323e-17 4.20935e-14 -1.71018e-46"/>
-            <geometry>
-                <mesh filename="package://legged_perceptive_description/urdf/nuc_and_lidar/mid_360_lidar_unit.stl"/>
+            <origin xyz="0.0240064 0.0460004 0.106664" rpy="6.12323e-17 -0.383972 -6.93889e-18"/>
+            <geometry>
+                <mesh filename="file://$(find legged_perceptive_description)/urdf/nuc_and_lidar/mid_360_lidar_unit.stl"/>
             </geometry>
         </collision>
@@ -45,5 +28,5 @@
             <origin xyz="0.1705 0.046 0.049" rpy="1.01161e-46 -2.30521e-16 -3.14159"/>
             <geometry>
-                <mesh filename="package://legged_perceptive_description/urdf/nuc_and_lidar/voltageregulatormount.stl"/>
+                <mesh filename="file://$(find legged_perceptive_description)/urdf/nuc_and_lidar/voltageregulatormount.stl"/>
             </geometry>
             <material name="voltageregulatormount_material">
@@ -54,5 +37,5 @@
             <origin xyz="0.1705 0.046 0.049" rpy="1.01161e-46 -2.30521e-16 -3.14159"/>
             <geometry>
-                <mesh filename="package://legged_perceptive_description/urdf/nuc_and_lidar/voltageregulatormount.stl"/>
+                <mesh filename="file://$(find legged_perceptive_description)/urdf/nuc_and_lidar/voltageregulatormount.stl"/>
             </geometry>
         </collision>
@@ -61,5 +44,5 @@
             <origin xyz="0.044 0.046 0.05" rpy="3.14159 -0 -1.5708"/>
             <geometry>
-                <mesh filename="package://legged_perceptive_description/urdf/nuc_and_lidar/nuc.stl"/>
+                <mesh filename="file://$(find legged_perceptive_description)/urdf/nuc_and_lidar/nuc.stl"/>
             </geometry>
             <material name="nuc_material">
@@ -70,5 +53,5 @@
             <origin xyz="0.044 0.046 0.05" rpy="3.14159 -0 -1.5708"/>
             <geometry>
-                <mesh filename="package://legged_perceptive_description/urdf/nuc_and_lidar/nuc.stl"/>
+                <mesh filename="file://$(find legged_perceptive_description)/urdf/nuc_and_lidar/nuc.stl"/>
             </geometry>
         </collision>
@@ -77,5 +60,5 @@
             <origin xyz="0.1175 0.092 -2.60209e-18" rpy="0 -0 3.14159"/>
             <geometry>
-                <mesh filename="package://legged_perceptive_description/urdf/nuc_and_lidar/nuc_enclosure_side.stl"/>
+                <mesh filename="file://$(find legged_perceptive_description)/urdf/nuc_and_lidar/nuc_enclosure_side.stl"/>
             </geometry>
             <material name="nuc_enclosure_side_material">
@@ -86,5 +69,5 @@
             <origin xyz="0.1175 0.092 -2.60209e-18" rpy="0 -0 3.14159"/>
             <geometry>
-                <mesh filename="package://legged_perceptive_description/urdf/nuc_and_lidar/nuc_enclosure_side.stl"/>
+                <mesh filename="file://$(find legged_perceptive_description)/urdf/nuc_and_lidar/nuc_enclosure_side.stl"/>
             </geometry>
         </collision>
@@ -93,5 +76,5 @@
             <origin xyz="-0.0305 5.58794e-11 0" rpy="0 -0 0"/>
             <geometry>
-                <mesh filename="package://legged_perceptive_description/urdf/nuc_and_lidar/nuc_enclosure_side.stl"/>
+                <mesh filename="file://$(find legged_perceptive_description)/urdf/nuc_and_lidar/nuc_enclosure_side.stl"/>
             </geometry>
             <material name="nuc_enclosure_side_2_material">
@@ -102,5 +85,5 @@
             <origin xyz="-0.0305 5.58794e-11 0" rpy="0 -0 0"/>
             <geometry>
-                <mesh filename="package://legged_perceptive_description/urdf/nuc_and_lidar/nuc_enclosure_side.stl"/>
+                <mesh filename="file://$(find legged_perceptive_description)/urdf/nuc_and_lidar/nuc_enclosure_side.stl"/>
             </geometry>
         </collision>
@@ -109,5 +92,5 @@
             <origin xyz="0.10975 0.0745 -2.60209e-18" rpy="-6.16298e-33 -1.2326e-32 -2.77556e-17"/>
             <geometry>
-                <mesh filename="package://legged_perceptive_description/urdf/nuc_and_lidar/mounting_rail.stl"/>
+                <mesh filename="file://$(find legged_perceptive_description)/urdf/nuc_and_lidar/mounting_rail.stl"/>
             </geometry>
             <material name="mounting_rail_material">
@@ -118,5 +101,5 @@
             <origin xyz="0.10975 0.0745 -2.60209e-18" rpy="-6.16298e-33 -1.2326e-32 -2.77556e-17"/>
             <geometry>
-                <mesh filename="package://legged_perceptive_description/urdf/nuc_and_lidar/mounting_rail.stl"/>
+                <mesh filename="file://$(find legged_perceptive_description)/urdf/nuc_and_lidar/mounting_rail.stl"/>
             </geometry>
         </collision>
@@ -125,5 +108,5 @@
             <origin xyz="0.169134 0.046 0.063" rpy="-2.30521e-16 -1.01161e-46 -1.5708"/>
             <geometry>
-                <mesh filename="package://legged_perceptive_description/urdf/nuc_and_lidar/psu.stl"/>
+                <mesh filename="file://$(find legged_perceptive_description)/urdf/nuc_and_lidar/psu.stl"/>
             </geometry>
             <material name="psu_material">
@@ -134,5 +117,5 @@
             <origin xyz="0.169134 0.046 0.063" rpy="-2.30521e-16 -1.01161e-46 -1.5708"/>
             <geometry>
-                <mesh filename="package://legged_perceptive_description/urdf/nuc_and_lidar/psu.stl"/>
+                <mesh filename="file://$(find legged_perceptive_description)/urdf/nuc_and_lidar/psu.stl"/>
             </geometry>
         </collision>
@@ -141,5 +124,5 @@
             <origin xyz="0.1725 0.008 0.026" rpy="-1.5708 2.30521e-16 0"/>
             <geometry>
-                <mesh filename="package://legged_perceptive_description/urdf/nuc_and_lidar/battery.stl"/>
+                <mesh filename="file://$(find legged_perceptive_description)/urdf/nuc_and_lidar/battery.stl"/>
             </geometry>
             <material name="battery_material">
@@ -150,12 +133,12 @@
             <origin xyz="0.1725 0.008 0.026" rpy="-1.5708 2.30521e-16 0"/>
             <geometry>
-                <mesh filename="package://legged_perceptive_description/urdf/nuc_and_lidar/battery.stl"/>
+                <mesh filename="file://$(find legged_perceptive_description)/urdf/nuc_and_lidar/battery.stl"/>
             </geometry>
         </collision>
         <!-- Part frame -->
         <visual>
-            <origin xyz="0.027 0.0460605 0.1336" rpy="-3.14159 2.43709e-17 3.14159"/>
-            <geometry>
-                <mesh filename="package://legged_perceptive_description/urdf/nuc_and_lidar/frame.stl"/>
+            <origin xyz="0.0045316 0.0460605 0.154866" rpy="3.14159 0.383972 3.14159"/>
+            <geometry>
+                <mesh filename="file://$(find legged_perceptive_description)/urdf/nuc_and_lidar/frame.stl"/>
             </geometry>
             <material name="frame_material">
@@ -164,7 +147,7 @@
         </visual>
         <collision>
-            <origin xyz="0.027 0.0460605 0.1336" rpy="-3.14159 2.43709e-17 3.14159"/>
-            <geometry>
-                <mesh filename="package://legged_perceptive_description/urdf/nuc_and_lidar/frame.stl"/>
+            <origin xyz="0.0045316 0.0460605 0.154866" rpy="3.14159 0.383972 3.14159"/>
+            <geometry>
+                <mesh filename="file://$(find legged_perceptive_description)/urdf/nuc_and_lidar/frame.stl"/>
             </geometry>
         </collision>
@@ -173,5 +156,5 @@
             <origin xyz="0.10975 -0.0175 0" rpy="0 -0 0"/>
             <geometry>
-                <mesh filename="package://legged_perceptive_description/urdf/nuc_and_lidar/mounting_rail.stl"/>
+                <mesh filename="file://$(find legged_perceptive_description)/urdf/nuc_and_lidar/mounting_rail.stl"/>
             </geometry>
             <material name="mounting_rail_2_material">
@@ -182,5 +165,21 @@
             <origin xyz="0.10975 -0.0175 0" rpy="0 -0 0"/>
             <geometry>
-                <mesh filename="package://legged_perceptive_description/urdf/nuc_and_lidar/mounting_rail.stl"/>
+                <mesh filename="file://$(find legged_perceptive_description)/urdf/nuc_and_lidar/mounting_rail.stl"/>
+            </geometry>
+        </collision>
+        <!-- Part part_1 -->
+        <visual>
+            <origin xyz="0.0435 0.0745 0.0515" rpy="3.14159 1.15074e-31 3.14159"/>
+            <geometry>
+                <mesh filename="file://$(find legged_perceptive_description)/urdf/nuc_and_lidar/part_1.stl"/>
+            </geometry>
+            <material name="part_1_material">
+                <color rgba="0.615686 0.811765 0.929412 1.0"/>
+            </material>
+        </visual>
+        <collision>
+            <origin xyz="0.0435 0.0745 0.0515" rpy="3.14159 1.15074e-31 3.14159"/>
+            <geometry>
+                <mesh filename="file://$(find legged_perceptive_description)/urdf/nuc_and_lidar/part_1.stl"/>
             </geometry>
         </collision>
@@ -189,5 +188,5 @@
             <origin xyz="0.1745 0.046 -6.93889e-18" rpy="-2.30521e-16 -0 -1.5708"/>
             <geometry>
-                <mesh filename="package://legged_perceptive_description/urdf/nuc_and_lidar/batterymount.stl"/>
+                <mesh filename="file://$(find legged_perceptive_description)/urdf/nuc_and_lidar/batterymount.stl"/>
             </geometry>
             <material name="batterymount_material">
@@ -198,22 +197,21 @@
             <origin xyz="0.1745 0.046 -6.93889e-18" rpy="-2.30521e-16 -0 -1.5708"/>
             <geometry>
-                <mesh filename="package://legged_perceptive_description/urdf/nuc_and_lidar/batterymount.stl"/>
+                <mesh filename="file://$(find legged_perceptive_description)/urdf/nuc_and_lidar/batterymount.stl"/>
             </geometry>
         </collision>
     </link>
-    <!-- Frame livox (dummy link + fixed joint) -->
-    <link name="livox">
-        <origin xyz="0 0 0" rpy="0 -0 0"/>
-        <inertial>
-            <origin xyz="0 0 0" rpy="0 0 0"/>
-            <mass value="1e-9"/>
-            <inertia ixx="0" ixy="0" ixz="0" iyy="0" iyz="0" izz="0"/>
-        </inertial>
-    </link>
-    <joint name="livox_frame" type="fixed">
-        <origin xyz="0.027 0.0460605 0.1336" rpy="-3.14159 2.43709e-17 3.14159"/>
-        <parent link="mid-360_lidar_unit"/>
-        <child link="livox"/>
-        <axis xyz="0 0 0"/>
+    <!-- Frame livox -->
+    <link name="lidar_frame"/>
+    <joint name="lidar_frame_joint" type="fixed">
+        <parent link="nuc_top"/>
+        <child link="lidar_frame"/>
+        <origin xyz="0.0045316 0.0460605 0.154866" rpy="0 0.383972 3.14159"/>
+    </joint>
+    <link name="lidar_imu_frame"/>
+    <joint name="lidar_imu_joint" type="fixed">
+        <parent link="lidar_frame"/>
+        <child link="lidar_imu_frame"/>
+        <!-- Extrinsics: translation from lidar_frame and identity rotation -->
+        <origin xyz="0.011 0.02329 -0.04412" rpy="0 0 0"/>
     </joint>
 </robot>

File: legged_perceptive_description/urdf/robot.xacro (robot description, xacro)
@@ -6,7 +6,7 @@
     <!-- <xacro:include filename="$(find legged_perceptive_description)/urdf/sensor_t265.xacro"/> -->
     <xacro:include filename="$(find legged_perceptive_description)/urdf/sensor_mid360.xacro"/>
-    <xacro:include filename="$(find legged_perceptive_description)/urdf/nuc_and_lidar/nuc_and_lidar.xacro"/>
+    <xacro:include filename="$(find legged_perceptive_description)/urdf/nuc_and_lidar/nuc_and_lidar_2.xacro"/>
     <xacro:sensor_d435 name="front_camera" topics_ns="front_camera" parent="base" sim="true">
-           <origin xyz="0.2844 -0.0 0.09" rpy="0 0.83 0"/>
+           <origin xyz="0.2844 -0.0 0.075" rpy="0 0.83 0"/>
       </xacro:sensor_d435>
     <!-- <xacro:sensor_t265 name="tracking_camera" topics_ns="tracking_camera" parent="base">
