Commit message: updated lidar frame pos

File: legged_perceptive_description/urdf/nuc_and_lidar/robot.urdf (robot description, URDF)
Before this commit: robot onshape, 3 links, 2 joints
Links:
- removed link lidar_frame
- removed link lidar_imu_frame
- removed link nuc_top
- added link livox, mass 1e-9
- added link mid-360_lidar_unit, mass 1.44797; collision mesh filename=package://legged_perceptive_description/urdf/nuc_and_lidar/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; collision mesh filename=package://legged_perceptive_description/urdf/nuc_and_lidar/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
Joints:
- removed joint lidar_frame_joint
- removed joint lidar_imu_joint
- added joint livox_frame: type fixed, parent mid-360_lidar_unit, child livox, origin xyz=0.00640463 0.0460605 0.15023 rpy=3.14159 0.383972 -3.14159, axis 0 0 0
